File: Subsystems/Electronics/Testing/Filters/ElectricalDesign/FilterTestBoard.brd (EAGLE design)
At the start: 160 x 100 mm, 21 parts

Commit message: Laid out Board
Parts:
- moved R3 100.4 mm to (47.0, 27.0), turned to 180 degrees
- moved R4 100.2 mm to (43.0, 27.0), turned to 180 degrees
- moved J2 94.8 mm to (54.0, 25.0), turned to 270 degrees
- moved C1 91.4 mm to (38.0, 40.0), turned to 270 degrees
- moved R1 81.7 mm to (39.0, 43.0), turned to 180 degrees
- moved R2 81.6 mm to (35.0, 43.0), turned to 180 degrees
- moved C5 78.8 mm to (39.0, 11.0), turned to 180 degrees
- moved C6 78.7 mm to (35.0, 11.0), turned to 180 degrees
- moved C7 78.3 mm to (39.0, 27.0), turned to 180 degrees
- moved C8 78.1 mm to (35.0, 27.0), turned to 180 degrees
- moved SW3 78.0 mm to (25.0, 9.00), turned to 90 degrees
- moved R5 73.3 mm to (38.0, 8.00), turned to 90 degrees
- moved R6 73.2 mm to (34.0, 8.00), turned to 90 degrees
- moved C3 71.9 mm to (46.0, 24.0), turned to 270 degrees
- moved C4 71.7 mm to (42.0, 24.0), turned to 270 degrees
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Connections:
- net N$1 renamed LOW_INT
- net N$10 renamed BAND_INT1
- net N$11 renamed LOW_IN
- net N$12 renamed HIGH_OUT
- net N$13 renamed HIGH_INT
- net N$14 renamed INPUT
- net N$15 renamed OUTPUT
- net N$2 renamed LOW_OUT
- net N$3 renamed BAND_OUT
- net N$4 renamed HIGH_IN
- net N$7 renamed BAND_INT2
- net N$8 renamed BAND_INT0
- net N$9 renamed BAND_IN
Routing:
- net PGND: track 0.00 -> 89.3 mm, vias 0 -> 4
- net INPUT: track 0.00 -> 67.3 mm
- net OUTPUT: track 0.00 -> 66.1 mm
- net BAND_IN: track 0.00 -> 31.1 mm
- net LOW_IN: track 0.00 -> 23.1 mm
- net HIGH_IN: track 0.00 -> 23.1 mm
- net HIGH_OUT: track 0.00 -> 17.2 mm
- net BAND_OUT: track 0.00 -> 17.2 mm
- net LOW_OUT: track 0.00 -> 17.2 mm
- net BAND_INT2: track 0.00 -> 4.46 mm
- net BAND_INT1: track 0.00 -> 4.46 mm
- net BAND_INT0: track 0.00 -> 4.46 mm
- net HIGH_INT: track 0.00 -> 4.46 mm
- net LOW_INT: track 0.00 -> 4.46 mm
Other:
- board size 160 x 100 mm -> 66 x 46 mm

Commit message: Changed Routing
Parts:
- moved C1 2.00 mm to (38.0, 38.0)
- moved C2 2.00 mm to (34.0, 38.0)
- moved C3 2.00 mm to (46.0, 22.0)
- moved C4 2.00 mm to (42.0, 22.0)
- moved C5 2.00 mm to (39.0, 9.00)
- moved C6 2.00 mm to (35.0, 9.00)
- moved C7 2.00 mm to (39.0, 25.0)
- moved C8 2.00 mm to (35.0, 25.0)
- moved J1 2.00 mm to (12.0, 23.0)
- moved J2 2.00 mm to (54.0, 23.0)
- moved R1 2.00 mm to (39.0, 41.0)
- moved R2 2.00 mm to (35.0, 41.0)
- moved R3 2.00 mm to (47.0, 25.0)
- moved R4 2.00 mm to (43.0, 25.0)
- moved R5 2.00 mm to (38.0, 6.00)
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Routing:
- net INPUT: track 67.3 -> 62.0 mm
- net HIGH_IN: track 23.1 -> 21.5 mm
- net BAND_IN: track 31.1 -> 29.7 mm
- net LOW_IN: track 23.1 -> 21.7 mm
- net PGND: track 89.3 -> 90.2 mm, vias 4 -> 1
- net OUTPUT: track 66.1 -> 65.6 mm

Commit message: Adjusted Board Layout
Connections:
- net INPUT: now also SW1.COM-B, SW2.COM-B, SW3.COM-B; no longer SW1.COM-A, SW2.COM-A, SW3.COM-A
- net OUTPUT: now also SW1.COM-A, SW2.COM-A, SW3.COM-A; no longer SW1.COM-B, SW2.COM-B, SW3.COM-B
Routing:
- net INPUT: track 62.0 -> 46.7 mm
- net OUTPUT: track 65.6 -> 62.9 mm
- net PGND: vias 1 -> 0
Changed lines of the file:
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@@
 <contactref element="R7" pad="1"/>
 <contactref element="R8" pad="1"/>
-<wire x1="12" y1="20.46" x2="14.54" y2="20.46" width="0.5" layer="16"/>
-<wire x1="17" y1="18" x2="25" y2="18" width="0.5" layer="16"/>
-<via x="25" y="18" extent="1-16" drill="0.35"/>
-<wire x1="14.54" y1="20.46" x2="17" y2="18" width="0.5" layer="16"/>
 <wire x1="34" y1="21.135" x2="38" y2="21.135" width="0.5" layer="1"/>
 <wire x1="38" y1="21.135" x2="42" y2="21.135" width="0.5" layer="1"/>
@@
 <wire x1="32.5" y1="20.5" x2="33.135" y2="21.135" width="0.5" layer="1"/>
 <wire x1="33.135" y1="21.135" x2="34" y2="21.135" width="0.5" layer="1"/>
-<wire x1="25" y1="18" x2="31" y2="18" width="0.5" layer="1"/>
+<wire x1="31" y1="18" x2="25" y2="18" width="0.5" layer="1"/>
 <wire x1="32.5" y1="19.5" x2="32.5" y2="20.5" width="0.5" layer="1"/>
-<wire x1="31" y1="18" x2="32.5" y2="19.5" width="0.5" layer="1"/>
+<wire x1="32.5" y1="19.5" x2="31" y2="18" width="0.5" layer="1"/>
 <wire x1="38" y1="5.135" x2="38.385" y2="5.135" width="0.5" layer="1"/>
 <wire x1="42" y1="8.75" x2="42" y2="21.135" width="0.5" layer="1"/>
@@
 <wire x1="50.79" y1="25.54" x2="39.195" y2="37.135" width="0.5" layer="1"/>
 <wire x1="39.195" y1="37.135" x2="38" y2="37.135" width="0.5" layer="1"/>
+<wire x1="25" y1="18" x2="17" y2="18" width="0.5" layer="1"/>
+<wire x1="17" y1="18" x2="14.54" y2="20.46" width="0.5" layer="1"/>
+<wire x1="14.54" y1="20.46" x2="12" y2="20.46" width="0.5" layer="1"/>
 </signal>
 <signal name="BAND_OUT">
@@
 <signal name="INPUT">
 <contactref element="J1" pad="CENTER"/>
-<contactref element="SW1" pad="COM-A"/>
-<contactref element="SW2" pad="COM-A"/>
-<contactref element="SW3" pad="COM-A"/>
-<wire x1="12" y1="23" x2="16" y2="23" width="0.5" layer="1"/>
-<wire x1="16" y1="30" x2="18" y2="32" width="0.5" layer="1"/>
-<wire x1="18" y1="32" x2="22" y2="32" width="0.5" layer="1"/>
-<wire x1="25" y1="35" x2="25" y2="36.59" width="0.5" layer="1"/>
-<wire x1="22" y1="32" x2="25" y2="35" width="0.5" layer="1"/>
-<wire x1="16" y1="23" x2="16" y2="18.5" width="0.5" layer="1"/>
-<wire x1="16" y1="23" x2="16" y2="30" width="0.5" layer="1"/>
-<wire x1="25" y1="20.59" x2="22.91" y2="18.5" width="0.5" layer="1"/>
-<wire x1="22.91" y1="18.5" x2="16" y2="18.5" width="0.5" layer="1"/>
-<wire x1="25" y1="4.59" x2="22.91" y2="2.5" width="0.5" layer="1"/>
-<wire x1="22.91" y1="2.5" x2="19.25" y2="2.5" width="0.5" layer="1"/>
-<wire x1="19.25" y1="2.5" x2="16" y2="5.75" width="0.5" layer="1"/>
-<wire x1="16" y1="5.75" x2="16" y2="18.5" width="0.5" layer="1"/>
+<contactref element="SW3" pad="COM-B"/>
+<contactref element="SW2" pad="COM-B"/>
+<contactref element="SW1" pad="COM-B"/>
+<wire x1="12" y1="23" x2="23" y2="23" width="0.5" layer="16"/>
+<wire x1="23" y1="23" x2="23" y2="25" width="0.5" layer="16"/>
+<wire x1="23" y1="25.41" x2="23" y2="39.41" width="0.5" layer="16"/>
+<wire x1="23" y1="39.41" x2="25" y2="41.41" width="0.5" layer="16"/>
+<wire x1="23" y1="23" x2="23" y2="11.41" width="0.5" layer="16"/>
+<wire x1="23" y1="11.41" x2="25" y2="9.41" width="0.5" layer="16"/>
+<wire x1="25" y1="25.41" x2="23" y2="25.41" width="0.5" layer="16"/>
+<wire x1="23" y1="25.41" x2="23" y2="25" width="0.5" layer="16"/>
 </signal>
 <signal name="OUTPUT">
+<contactref element="SW3" pad="COM-A"/>
+<contactref element="SW2" pad="COM-A"/>
+<contactref element="SW1" pad="COM-A"/>
 <contactref element="J2" pad="CENTER"/>
-<contactref element="SW2" pad="COM-B"/>
-<contactref element="SW3" pad="COM-B"/>
-<contactref element="SW1" pad="COM-B"/>
-<wire x1="54" y1="23" x2="47" y2="30" width="0.5" layer="16"/>
-<wire x1="27" y1="25.41" x2="25" y2="25.41" width="0.5" layer="16"/>
-<wire x1="27" y1="30" x2="27" y2="25.41" width="0.5" layer="16"/>
-<wire x1="47" y1="30" x2="27" y2="30" width="0.5" layer="16"/>
-<wire x1="27" y1="30" x2="27" y2="39.41" width="0.5" layer="16"/>
-<wire x1="27" y1="39.41" x2="25" y2="41.41" width="0.5" layer="16"/>
-<wire x1="27" y1="25.41" x2="27" y2="11.41" width="0.5" layer="16"/>
-<wire x1="27" y1="11.41" x2="25" y2="9.41" width="0.5" layer="16"/>
+<wire x1="25" y1="4.59" x2="27.25" y2="6.84" width="0.5" layer="16"/>
+<wire x1="27.25" y1="34.34" x2="25" y2="36.59" width="0.5" layer="16"/>
+<wire x1="27.25" y1="6.84" x2="27.25" y2="20.59" width="0.5" layer="16"/>
+<wire x1="27.25" y1="20.59" x2="27.25" y2="23" width="0.5" layer="16"/>
+<wire x1="27.25" y1="23" x2="27.25" y2="34.34" width="0.5" layer="16"/>
+<wire x1="25" y1="20.59" x2="27.25" y2="20.59" width="0.5" layer="16"/>
+<wire x1="54" y1="23" x2="27.25" y2="23" width="0.5" layer="16"/>
 </signal>
 </signals>
