File: Subsystems/Electronics/Testing/Filters/ElectricalDesign/FilterTestBoard.brd (EAGLE design)
At the start: 66 x 46 mm, 21 parts

Commit message: Exported Schematics
Parts:
- C1, C2, C3, C4, C5, C6, C7, C8: value 1nF 10% -> 10µF 10%
- R1, R2, R7, R8: value 0Ω <20mΩ -> 158kΩ 0.1%
- R3, R4, R5, R6: value 0Ω <20mΩ -> 158Ω 1%
