File: Subsystems/Electronics/Testing/SolarSimulator/ElectricalDesign/UTJ-1.sch (EAGLE design)
At the start: 10 parts, among them Q1 2N2219A, Q2 2N2219A, Q3 2N2219A, Q4 2N2219A, Q5 2N2219A

Commit message: Laid out solar simulator
Parts:
- added LOGO1: SIGNATUREBRADLEY, CougsInSpace-Aesthetics:SIGNATUREBRADLEY
Connections:
- net N$1 renamed EMITTER-1
- net N$2 renamed EMITTER-2
- net N$3 renamed CELL+
- net N$4 renamed PGND
- net N$5 renamed ZENER_C
Changed lines of the file:
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@@
 <part name="H1" library="CougsInSpace-Hardware" deviceset="MOUNTING_HOLE" device="-6.6" value="M6"/>
 <part name="H2" library="CougsInSpace-Hardware" deviceset="MOUNTING_HOLE" device="-6.6" value="M6"/>
+<part name="SUPPLY1" library="CougsInSpace-PowerSymbols" deviceset="PGND" device=""/>
+<part name="LOGO1" library="CougsInSpace-Aesthetics" deviceset="SIGNATURE" device="BRADLEY"/>
 </parts>
 <sheets>
@@
 <attribute name="SKU" x="86.36" y="68.834" size="1.27" layer="97" rot="MR0" align="center"/>
 </instance>
+<instance part="SUPPLY1" gate="G$1" x="93.98" y="68.58" smashed="yes"/>
+<instance part="LOGO1" gate="G$1" x="10.16" y="5.08" smashed="yes">
+<attribute name="NAME" x="10.16" y="7.874" size="1.778" layer="95" align="bottom-center"/>
+</instance>
 </instances>
 <busses>
 </busses>
 <nets>
-<net name="N$1" class="0">
+<net name="EMITTER-1" class="0">
 <segment>
 <pinref part="Q5" gate="G$1" pin="E"/>
@@
 </segment>
 </net>
-<net name="N$2" class="0">
+<net name="EMITTER-2" class="0">
 <segment>
 <pinref part="Q4" gate="G$1" pin="E"/>
@@
 </segment>
 </net>
-<net name="N$3" class="0">
+<net name="CELL+" class="0">
 <segment>
 <pinref part="Q3" gate="G$1" pin="C"/>
@@
 </segment>
 </net>
-<net name="N$4" class="0">
+<net name="ZENER_C" class="0">
+<segment>
+<pinref part="Q5" gate="G$1" pin="B"/>
+<pinref part="D1" gate="G$1" pin="C"/>
+<wire x1="132.08" y1="104.14" x2="121.92" y2="104.14" width="0.1524" layer="91"/>
+<wire x1="121.92" y1="104.14" x2="121.92" y2="109.22" width="0.1524" layer="91"/>
+<pinref part="R1" gate="G$1" pin="2"/>
+<wire x1="121.92" y1="83.82" x2="121.92" y2="104.14" width="0.1524" layer="91"/>
+<junction x="121.92" y="104.14"/>
+</segment>
+</net>
+<net name="PGND" class="0">
 <segment>
 <pinref part="Q1" gate="G$1" pin="E"/>
@@
 <wire x1="111.76" y1="73.66" x2="111.76" y2="76.2" width="0.1524" layer="91"/>
 <junction x="121.92" y="73.66"/>
-<wire x1="111.76" y1="73.66" x2="88.9" y2="73.66" width="0.1524" layer="91"/>
+<wire x1="111.76" y1="73.66" x2="93.98" y2="73.66" width="0.1524" layer="91"/>
 <junction x="111.76" y="73.66"/>
 <pinref part="H2" gate="G$1" pin="MOUNT"/>
-</segment>
-</net>
-<net name="N$5" class="0">
-<segment>
-<pinref part="Q5" gate="G$1" pin="B"/>
-<pinref part="D1" gate="G$1" pin="C"/>
-<wire x1="132.08" y1="104.14" x2="121.92" y2="104.14" width="0.1524" layer="91"/>
-<wire x1="121.92" y1="104.14" x2="121.92" y2="109.22" width="0.1524" layer="91"/>
-<pinref part="R1" gate="G$1" pin="2"/>
-<wire x1="121.92" y1="83.82" x2="121.92" y2="104.14" width="0.1524" layer="91"/>
-<junction x="121.92" y="104.14"/>
-</segment>
-</net>
+<pinref part="SUPPLY1" gate="G$1" pin="PGND"/>
+<wire x1="93.98" y1="73.66" x2="88.9" y2="73.66" width="0.1524" layer="91"/>
+<wire x1="93.98" y1="71.12" x2="93.98" y2="73.66" width="0.1524" layer="91"/>
+<junction x="93.98" y="73.66"/>
+</segment>
+</net>
