File: Subsystems/Electronics/Testing/SolarSimulator/ElectricalDesign/UTJ.brd (EAGLE design)
At the start: 32 x 35.5 mm, 11 parts, among them Q1 2N2219A, Q2 2N2219A, Q3 2N2219A, Q4 2N2219A, Q5 2N2219A

Commit message: Exported Gerbers
Parts:
- moved LOGO1 14.8 mm to (0.00, 26.3)
- moved Q1 2.01 mm to (10.8, 11.0)
- moved Q3 2.01 mm to (-10.8, 11.0), turned to 270 degrees
- moved D1 1.22 mm to (-2.00, 15.4)
- moved R1 1.22 mm to (1.80, 15.4)
- moved Q4 0.63 mm to (-6.60, 21.6), turned to 315 degrees
- moved Q5 0.63 mm to (6.60, 21.6), turned to 45 degrees
- turned Q2 to 180 degrees
Routing:
- net PGND: track 111.8 -> 137.4 mm
- net CELL+: track 137.0 -> 153.1 mm
- net ZENER_C: track 13.7 -> 18.2 mm
- net EMITTER-1: track 12.0 -> 14.4 mm
- net EMITTER-2: track 65.9 -> 64.7 mm
Other:
- board text added: "MAX 600mA 100%=453mA"
- board text removed: "MAX 600mA UTJ = 453mA"
