File: Subsystems/Electronics/Testing/ElectronicLoad/ElectricalDesign/ElectronicLoad.sch (EAGLE design)
At the start: 8 parts, among them Q1 2N2219A, SW1 D2MQ-1-TL, SW2 D2MQ-1-TL, SW3 D2MQ-1-TL, SW4 D2MQ-1-TL, U1 STM32L432KCU

Commit message: Update ElectronicLoad.sch
Parts:
- removed DS1: Blue, CougsInSpace-LEDs:LED-H-BLU-1608
- removed SW1, SW2, SW3, SW4: D2MQ-1-TL, CougsInSpace-Switches:SWITCH-SPDT-D2MQ-1-TL
- added C1, C10, C11, C2, C3, C6: 100nF 10%, CougsInSpace-Capacitors:CAP-V-100NF-1608
- added C4, C5: 47pF 5%, CougsInSpace-Capacitors:CAP-V-47PF-1608
- added C7: 10nF 10%, CougsInSpace-Capacitors:CAP-V-10NF-1608
- added C8: 4.7µF 10%, CougsInSpace-Capacitors:CAP-POL-V-4.7UF-4028
- added C9: 100nF 10%, CougsInSpace-Capacitors:CAP-H-100NF-1608
- added DS3: Green, CougsInSpace-LEDs:LED-V-GRN-1608
- added DS5: Red, CougsInSpace-LEDs:LED-V-RED-1608
- added FB1: 1.5kΩ @ 100MHz, CougsInSpace-Coils:CHOKE-H-1.5K-1608
- added J2: Current Input, CougsInSpace-Connectors:1X02-TERMINAL-SPRING-02
- added J3: Current Sense, CougsInSpace-Connectors:1X02-TERMINAL-SPRING-02
- added J4: Voltage Sense, CougsInSpace-Connectors:1X03-TERMINAL-SPRING-3
- added Q2, Q3: SiRA20DP, CougsInSpace-DiscreteSemi:MOSFET-N-SIRA20DP-POWERPAK-SO8
- added Q4: IRFP4368PBF, CougsInSpace-DiscreteSemi:MOSFET-N-IRFP4368PBF-TO247-3-DOWN
- added R1: 50mΩ 1%, CougsInSpace-Resistors:RES-V-0.05R-1608
- added R13, R15: 1kΩ 0.1%, CougsInSpace-Resistors:RES-H-1K-1608
- added R2, R6: 5mΩ 1%, CougsInSpace-Resistors:RES-V-KELVIN-0.005R-1632
- added R3, R4: 27Ω 1%, CougsInSpace-Resistors:RES-H-27R-1608
- added R5: 510mΩ 1%, CougsInSpace-Resistors:RES-V-0.51R-1608
- added R7: 10kΩ 0.1%, CougsInSpace-Resistors:RES-H-10K-1608
- added R8: 47kΩ 0.1%, CougsInSpace-Resistors:RES-V-47K-1608
- added R9: 1kΩ 0.1%, CougsInSpace-Resistors:RES-V-1K-1608
- added RN1: 10kΩ 1%, CougsInSpace-Resistors:RES-4-V-10K-1632
- added TP5, TP6: TEST_POINT-THT-1.0, CougsInSpace-Connectors:TEST_POINT-THT-1.0
- added U2: AD8515, CougsInSpace-IC-Amplifiers:OPAMP-1-AD8515
- added U3: FT230XQ, CougsInSpace-IC-Comms:FT230X-QFN16
- added U4, U6: INA199C1, CougsInSpace-IC-Amplifiers:INA199C1
- added U5: STM32L476RGT, CougsInSpace-IC-µController:STM32-64P-L476RGT
- J1: value (none) -> USB; device CougsInSpace-Connectors:1X04-PICOLOCK -> CougsInSpace-Connectors:USB-B-FEMALE
- Q1: value 2N2219A -> IRFP4368PBF; device CougsInSpace-DiscreteSemi:BJT-NPN-2N2219A-TO-39 -> CougsInSpace-DiscreteSemi:MOSFET-N-IRFP4368PBF-TO247-3-DOWN
- U1: value STM32L432KCU -> STM32L476RGT; device CougsInSpace-IC-µController:STM32-32P-L432KCU -> CougsInSpace-IC-µController:STM32-64P-L476RGT
Connections:
- removed net 9.0V: SW1.NO, SW2.NO, SW3.NO, SW4.NO
- removed net AGND: DS1.C, Q1.B, SW1.NC, SW2.NC, SW3.NC, SW4.NC
- removed net AVDD: J1.2
- removed net N$1: SW1.COM
- removed net N$2: SW2.COM
- removed net N$3: SW3.COM
- removed net N$4: SW4.COM
- removed net N$5: DS1.A
- removed net N$6: Q1.E
- removed net N$7: J1.1, Q1.C
- removed net N$8: J1.4
- removed net N$9: J1.3
- new net !CTS: RN1D.1, U3.!CTS
- new net !RTS: RN1C.1, U3.!RTS
- new net 3.3V: C3.1, DS3.A, DS5.A, R7.1, RN1A.2, RN1B.2, RN1C.2, RN1D.2, U3.3V3OUT, U3.VCCIO
- new net 5.0V: C1.1, C10.1, C11.1, C2.1, U2.V+, U4.VDD, U6.VDD
- new net 5.0V1: U1BASE.VDD@1, U1BASE.VDD@2, U1BASE.VDD@3
- new net CBUS1: R15.1, U3.CBUS1
- new net CBUS2: R13.1, U3.CBUS2
- new net CHASSIS: J1.SHIELD
- new net DAC_IN: R8.2, U5A.PA4
- new net DGND: C1.2, C10.2, C11.2, C2.2, C3.2, C4.2, C5.2, C6.2, C7.2, C8.C, C9.2, J1.GND, J4.3, R9.1, U2.V-, U3.DGND, U4.GND, U4.REF, U6.GND, U6.REF
- new net DGND1: U1BASE.VSS@1, U1BASE.VSS@2, U1BASE.VSS@3, U1BASE.VSS@4
- new net FEEDBACK: Q1.S, Q2.D, Q4.S, R5.2, U2.IN-
- new net FET_GATE: Q1.G, Q4.G, U2.OUT
- new net INPUT_SHUNT+: R2.2-KELVIN, U4.IN+
- new net INPUT_SHUNT-: R2.1-KELVIN, U4.IN-
- new net I_ADJUST_IN: R8.1, R9.2, U2.IN+
- new net I_IN: J2.1, Q1.D, Q4.D
- new net I_OUT: J2.2, R6.1
- new net I_SENSE_IN+: J3.1, R2.2, U4.OUT, U5C.PC0
- new net I_SENSE_IN-: J3.2, R2.1, U5C.PC2, U6.OUT
- new net OUTPUT_SHUNT+: R6.2-KELVIN, U6.IN+
- new net OUTPUT_SHUNT-: R6.1-KELVIN, U6.IN-
- new net RX: RN1A.1, U3.TXD, U5A.PA10
- new net RXLED_C: DS5.C, R13.2
- new net SHUNT_LOW: Q3.S, R1.1, R6.2
- new net SHUNT_MID: Q2.S, Q3.D, R1.2, R5.1
- new net TX: RN1B.1, U3.RXD, U5A.PA9
- new net TXLED_C: DS3.C, R15.2
- new net USB5V: C7.1, FB1.1, J1.VCC, TP5.1
- new net USB5V_FILTERED: C6.1, C8.A, FB1.2, TP6.1, U3.VCC
- new net USB_CONN_N: C4.1, J1.DATA_N, R4.1
- new net USB_CONN_P: C5.1, J1.DATA_P, R3.1
- new net USB_N: R4.2, U3.USBD_N
- new net USB_P: R3.2, U3.USBD_P
- new net USB_RESET: C9.1, R7.2, U3.!RESET
- new net V_SENSE_IN: J4.1, U5C.PC1
- new net V_SENSE_OUT: J4.2, U5C.PC3
Other:
- note added: "CAD Note: Decoupling"
- note removed: "Fan"

Commit message: Update ElectronicLoad.sch
Parts:
- added B1: 128x32p White on Blue, CougsInSpace-Boards:NHD-C12832A11Z-NSW-BBW-3V3
- added C12: 4.7µF 10%, CougsInSpace-Capacitors:CAP-POL-V-4.7UF-4028
- added C13: 100nF 10%, CougsInSpace-Capacitors:CAP-V-100NF-1608
- added DS1: Green, CougsInSpace-LEDs:LED-H-GRN-1608
- added FB2: 1.5kΩ @ 100MHz, CougsInSpace-Coils:CHOKE-H-1.5K-1608
- added J5: SWD, CougsInSpace-Connectors:SWDSMD-6-R
- added R10: 0Ω <20mΩ, CougsInSpace-Resistors:RES-H-0-1608
- added R11: 1kΩ 0.1%, CougsInSpace-Resistors:RES-V-1K-1608
- added TP1: TEST_POINT-SMD-C-1.25, CougsInSpace-Connectors:TEST_POINT-SMD-C-1.25
Connections:
- new net AGND: C12.C, C13.2, U1BASE.VSSA/VREF-
- new net AVDD: C12.A, C13.1, FB2.2, TP1.1, U1BASE.VDDA/VREF+
- new net BOOT0: R10.2, U1BASE.BOOT0
- new net FET_1_OUT: Q2.G, U5C.PC5
- new net FET_2_OUT: Q3.G, U5C.PC6
- new net JTAG_TCK: J5.SWCLK, U5A.PA14
- new net JTAG_TDI: J5.SWO, U5A.PA15
- new net JTAG_TMS: J5.SWDIO, U5A.PA13
- new net N$1: J5.VSENSE, R11.1
- new net NRST: J5.!RST, U1BASE.!NRST
- new net SWD_GROUND: J5.DGND
- new net TO_LED: DS1.A, U1BASE.EXTRA_PIN
- net 5.0V: now also FB2.1, R11.2
- net 5.0V1: now also U1BASE.VBAT, U1BASE.VDDUSB
- net DGND: now also DS1.C, R10.1
Other:
- note added: "1: Overview"
- note added: "2: Electroic Load Schematic"
- note added: "3: Microcontroller and USB Schematic"
- note added: "3B5>"
- note added: "<3B5"
- note added: "<A5"
- note added: "<B2"
- note added: "<B2>"
- note added: "<B4"
- note added: "<B5"
- note added: "<C5"
- note added: "<D2"
- note added: "<D5"
- note added: "<D5>"
- note added: "A3>"
- note added: "A6>"
- note added: "B2>"
- note added: "B4>"
- note added: "B5>"
- note added: "Page 2"
- note added: "Page 3"
- note removed: "Page x"
- moved on the sheet: C1, C10, C11, C2, C3, C4, C5, C6, C7, C8, C9, DS3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

Commit message: Update ElectronicLoad.sch
Parts:
- added C14, C15, C16, C17, C18, C21: 1µF 10%, CougsInSpace-Capacitors:CAP-H-1UF-1608
- added C19, C20: 1nF 1%, CougsInSpace-Capacitors:CAP-V-1NF-B-1608
Connections:
- removed net I_SENSE_IN+: J3.1, R2.2, U4.OUT, U5C.PC0
- new net A0_LCD: B1.A0, U5A.PA0
- new net CS_LCD: B1.!CS, U5A.PA2
- new net I_SENSE_IN: J3.1, R2.2, U4.OUT, U5C.PC0, U6.OUT
- new net N$10: B1.V3, C16.1
- new net N$11: B1.V4, C18.1
- new net N$2: B1.C1+, C20.1
- new net N$3: B1.C1-, C20.2
- new net N$4: B1.C2+, C19.1
- new net N$5: B1.C2-, C19.2
- new net N$6: B1.VOUT, C21.2
- new net N$7: B1.V0, C15.1
- new net N$8: B1.V1, C17.1
- new net N$9: B1.V2, C14.1
- new net RST_LCD: B1.!RST, U5A.PA1
- new net SPI_MOSI: B1.MOSI, U5A.PA7
- new net SPI_SCK: B1.SCK, U5A.PA5
- net AVDD: now also B1.LED+, B1.VDD
- net DGND: now also B1.LED-, B1.VSS, C14.2, C15.2, C16.2, C17.2, C18.2, C21.1
- net I_SENSE_IN-: no longer U6.OUT

Commit message: Update ElectronicLoad.sch
Other:
- note added: "<C2"
- moved on the sheet: B1, C1, C10, C11, C12, C13, C14, C15, C16, C17, C18, C19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

Commit message: Update ElectronicLoad.sch
Other:
- note added: "<A2"
- note added: "<A2>"
- note added: "<B1"
- note added: "<B6"
- note added: "<B6>"
- note added: "<C1"
- note added: "A2>"
- note added: "B3>"
- note added: "C2>"
- note added: "C3>"
- note added: "C4>"
- note added: "C5>"
- note removed: "3B5>"
- note removed: "<3B5"
- note removed: "<B2>"
- note removed: "<B4"
- note removed: "<D2"
- note removed: "<D5"
- note removed: "<D5>"
- note removed: "A3>"
- note removed: "A6>"
- note removed: "B4>"
- moved on the sheet: B1, C12, C13, C19, C20, C21, FB2, J5, R11, TP1, U5A, U5B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

Commit message: Update ElectronicLoad.sch
Parts:
- added SW1: [Override], CougsInSpace-Sensors:ENCODER-SW-PEC12R-4-S
- added SW2: [Override], CougsInSpace-Switches:SWITCH-SPST-NO-B3F-1050-THT-6060
Connections:
- net I_SENSE_IN renamed I_SENSE_OUT
- removed net N$7 (its old number): B1.V0, C15.1
- new net A_ENC: SW1.A, U5C.PC7
- new net B_ENC: SW1.B, U5C.PC8
- new net N$9: SW2.COM, U5C.PC11
- new net SW_C: SW1.SW-CM, U5C.PC10
- new net SW_N: SW1.SW-NO, U5C.PC9
- net AGND: now also SW1.CM
- net AVDD: now also SW1.SHIELD, SW2.NO
Other:
- note added: "3C5>"
- note added: "4B5>"
- note added: "<3A5"
- note added: "<3B1"
- note added: "<3B5"
- note added: "<3B6"
- note added: "<3C1"
- note added: "<4B5"
- note added: "<C4"
- note added: "<C6"
- note removed: "<A5"
- note removed: "<B1"
- note removed: "<C1"
- note removed: "B5>"
- moved on the sheet: C1, C10, C11, C12, C13, C14, C15, C16, C17, C18, C2, DS1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

Commit message: Update ElectronicLoad.sch
Parts:
- removed C18: 1µF 10%, CougsInSpace-Capacitors:CAP-H-1UF-1608
- added C22: 1µF 10%, CougsInSpace-Capacitors:CAP-V-1UF-B-1608
- added R12, R14: 10kΩ 0.1%, CougsInSpace-Resistors:RES-V-10K-1608
- C14, C15, C16, C17: device CougsInSpace-Capacitors:CAP-H-1UF-1608 -> CougsInSpace-Capacitors:CAP-V-1UF-B-1608
Connections:
- removed net SW_C: SW1.SW-CM, U5C.PC10
- new net N$12: B1.V0, C17.1
- new net N$13: SW2.NO
- net AGND: now also SW1.SHIELD, SW1.SW-CM
- net AVDD: now also R12.2, R14.2; no longer SW1.SHIELD, SW2.NO
- net A_ENC: now also R12.1
- net B_ENC: now also R14.1
- net DGND: now also B1.SHIELD, C22.2; no longer C18.2
- net N$10: now also C14.1; no longer C16.1
- net N$11: now also C22.1; no longer C18.1
- net N$7: now also C15.1; no longer C14.1
- net N$8: now also C16.1; no longer C17.1
Other:
- note added: "B5>"
- note removed: "<C4"
- moved on the sheet: SW1

Commit message: Electronic Load (Hopefully Im done now)
Parts:
- removed U5: STM32L476RGT, CougsInSpace-IC-µController:STM32-64P-L476RGT
- added C18, C23: 10pF 5%, CougsInSpace-Capacitors:CAP-V-10PF-1608
- added R16: 10kΩ 0.1%, CougsInSpace-Resistors:RES-V-10K-1608
- added R17: 0Ω <20mΩ, CougsInSpace-Resistors:RES-V-0-1608
- added Y1: 8MHz ±10ppm, CougsInSpace-Clocks:CRYSTAL-GROUNDED-8M-SMD-5032
- SW1: value [Override] -> Nice Knob
- SW2: value [Override] -> Nice Button
Connections:
- net I_ADJUST_IN renamed N$1
- net N$1 renamed VSENSE
- net N$10 renamed LCD_V3
- net N$11 renamed LCD_V4
- net N$12 renamed LCD_V0
- net N$2 renamed C1+
- net N$3 renamed C1-
- net N$4 renamed C2+
- net N$5 renamed C2-
- net N$6 renamed VOUT
- net N$7 renamed LCD_V2
- net N$8 renamed LCD_V1
- removed net 5.0V1: U1BASE.VBAT, U1BASE.VDD@1, U1BASE.VDD@2, U1BASE.VDD@3, U1BASE.VDDUSB
- removed net DGND1: U1BASE.VSS@1, U1BASE.VSS@2, U1BASE.VSS@3, U1BASE.VSS@4
- removed net N$13: SW2.NO
- removed net N$9: SW2.COM, U5C.PC11
- removed net SWD_GROUND: J5.DGND
- new net I_SENSE_IN: U1C.PC2, U4.OUT
- new net I_SENSE_IN+: J3.1, R2.2
- new net N$2: C23.1, U1BASE.PH0-OSC_IN, Y1.2
- new net N$3: C18.1, U1BASE.PH1-OSC_OUT, Y1.1
- new net NICE_BUTTON: R16.1, SW2.COM, U1C.PC11
- net 5.0V: now also U1BASE.VBAT, U1BASE.VDD@1, U1BASE.VDD@2, U1BASE.VDD@3, U1BASE.VDDUSB
- net A0_LCD: now also U1A.PA0; no longer U5A.PA0
- net AGND: no longer SW1.CM, SW1.SHIELD, SW1.SW-CM
- net AVDD: now also R16.2
- net A_ENC: now also U1C.PC7; no longer U5C.PC7
- net B_ENC: now also U1C.PC8; no longer U5C.PC8
- net CHASSIS: now also R17.2
- net CS_LCD: now also U1A.PA2; no longer U5A.PA2
- net DAC_IN: now also U1A.PA4; no longer U5A.PA4
- net DGND: now also C18.2, C23.2, J5.DGND, R17.1, SW1.CM, SW1.SHIELD, SW1.SW-CM, SW2.NO, U1BASE.VSS@1, U1BASE.VSS@2, U1BASE.VSS@3, U1BASE.VSS@4, Y1.GND
- net FET_1_OUT: now also U1C.PC5; no longer U5C.PC5
- net FET_2_OUT: now also U1C.PC6; no longer U5C.PC6
- net I_SENSE_IN-: no longer U5C.PC2
- net I_SENSE_OUT: now also U1C.PC0; no longer J3.1, R2.2, U4.OUT, U5C.PC0
- net JTAG_TCK: now also U1A.PA14; no longer U5A.PA14
- net JTAG_TDI: now also U1A.PA15; no longer U5A.PA15
- net JTAG_TMS: now also U1A.PA13; no longer U5A.PA13
- net RST_LCD: now also U1A.PA1; no longer U5A.PA1
- net RX: now also U1A.PA10; no longer U5A.PA10
- net SPI_MOSI: now also U1A.PA7; no longer U5A.PA7
- net SPI_SCK: now also U1A.PA5; no longer U5A.PA5
- net SW_N: now also U1C.PC9; no longer U5C.PC9
- net TX: now also U1A.PA9; no longer U5A.PA9
- net V_SENSE_IN: now also U1C.PC1; no longer U5C.PC1
- net V_SENSE_OUT: now also U1C.PC3; no longer U5C.PC3
Other:
- note added: "2A2>"
- note added: "2B2>"
- note added: "2B5>"
- note added: "2C2>"
- note added: "2C4>"
- note added: "2C5>"
- note added: "3B3>"
- note added: "3C3>"
- note added: "<2A2"
- note added: "<2A2>"
- note added: "<2B2"
- note added: "<2B6"
- note added: "<2B6>"
- note added: "<2C2"
- note added: "<2C5"
- note added: "<2C6"
- note removed: "<A2"
- note removed: "<A2>"
- note removed: "<B2"
- note removed: "<B5"
- note removed: "<B6"
- note removed: "<B6>"
- note removed: "<C2"
- note removed: "<C5"
- note removed: "<C6"
- note removed: "A2>"
- note removed: "B2>"
- note removed: "B3>"
- note removed: "B5>"
- note removed: "C2>"
- note removed: "C3>"
- note removed: "C4>"
- note removed: "C5>"
- moved on the sheet: DS3, DS5, SW2
