File: Subsystems/Electronics/Testing/ElectronicLoad/ElectricalDesign/ElectronicLoad.sch (EAGLE design)
At the start: 72 parts, among them J1 USB, J2 Current Input, J3 Current Sense, J4 Voltage Sense, J5 SWD, Q1 IRFP4368PBF, Q2 SiRA20DP, Q3 SiRA20DP, Q4 IRFP4368PBF, SW1 Nice Knob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

Commit message: Update ElectronicLoad.sch
Connections:
- net FAN_CONTROL: now also U1A.PA6
Changed lines of the file:
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@@
 <text x="228.6" y="154.94" size="1.778" layer="95" align="center-left"> &lt;2A2&gt;</text>
 <text x="228.6" y="149.86" size="1.778" layer="95" align="center-left"> &lt;2A2</text>
-<text x="55.88" y="60.96" size="1.778" layer="95" align="center-left"> &lt;2A6&gt;</text>
-<text x="55.88" y="58.42" size="1.778" layer="95" align="center-left"> &lt;2A6</text>
-<text x="55.88" y="55.88" size="1.778" layer="95" align="center-left"> &lt;2A6</text>
-<text x="55.88" y="71.12" size="1.778" layer="95" align="center-left"> 4B5&gt;</text>
-<text x="55.88" y="68.58" size="1.778" layer="95" align="center-left"> &lt;4B5</text>
-<text x="55.88" y="93.98" size="1.778" layer="95" align="center-left"> 3C5&gt;</text>
-<text x="55.88" y="91.44" size="1.778" layer="95" align="center-left"> 3C5&gt;</text>
-<text x="55.88" y="88.9" size="1.778" layer="95" align="center-left"> 3C5&gt;</text>
-<text x="55.88" y="81.28" size="1.778" layer="95" align="center-left"> 3C5&gt;</text>
-<text x="55.88" y="76.2" size="1.778" layer="95" align="center-left"> 3C5&gt;</text>
-<text x="55.88" y="83.82" size="1.778" layer="95" align="center-left"> 3B2&gt;</text>
+<text x="60.96" y="60.96" size="1.778" layer="95" align="center-left"> &lt;2A6&gt;</text>
+<text x="60.96" y="58.42" size="1.778" layer="95" align="center-left"> &lt;2A6</text>
+<text x="60.96" y="55.88" size="1.778" layer="95" align="center-left"> &lt;2A6</text>
+<text x="60.96" y="71.12" size="1.778" layer="95" align="center-left"> 4B5&gt;</text>
+<text x="60.96" y="68.58" size="1.778" layer="95" align="center-left"> &lt;4B5</text>
+<text x="60.96" y="93.98" size="1.778" layer="95" align="center-left"> 3C5&gt;</text>
+<text x="60.96" y="91.44" size="1.778" layer="95" align="center-left"> 3C5&gt;</text>
+<text x="60.96" y="88.9" size="1.778" layer="95" align="center-left"> 3C5&gt;</text>
+<text x="60.96" y="81.28" size="1.778" layer="95" align="center-left"> 3C5&gt;</text>
+<text x="60.96" y="76.2" size="1.778" layer="95" align="center-left"> 3C5&gt;</text>
+<text x="60.96" y="83.82" size="1.778" layer="95" align="center-left"> 3B2&gt;</text>
 <text x="139.7" y="93.98" size="1.778" layer="95" align="center-left"> &lt;3C3</text>
 <text x="139.7" y="91.44" size="1.778" layer="95" align="center-left"> &lt;3B5</text>
@@
 <wire x1="53.34" y1="162.56" x2="53.34" y2="185.42" width="0.1524" layer="97" style="shortdash"/>
 <text x="83.82" y="163.83" size="1.778" layer="97" align="center">CAD Note: Decoupling</text>
-<text x="55.88" y="66.04" size="1.778" layer="95" align="center-left"> 3A2&gt;</text>
+<text x="60.96" y="66.04" size="1.778" layer="95" align="center-left"> 3A2&gt;</text>
 </plain>
 <instances>
@@
 <attribute name="SKU" x="54.61" y="116.84" size="1.27" layer="97" align="center"/>
 </instance>
-<instance part="OFFSHEET3" gate="G$1" x="53.34" y="71.12" smashed="yes" rot="MR0"/>
-<instance part="OFFSHEET4" gate="G$1" x="53.34" y="68.58" smashed="yes" rot="MR0"/>
+<instance part="OFFSHEET3" gate="G$1" x="58.42" y="71.12" smashed="yes" rot="MR0"/>
+<instance part="OFFSHEET4" gate="G$1" x="58.42" y="68.58" smashed="yes" rot="MR0"/>
 <instance part="J5" gate="G$1" x="195.58" y="154.94" smashed="yes">
 <attribute name="VALUE" x="194.31" y="146.05" size="1.778" layer="96" align="center"/>
@@
 <instance part="OFFSHEET8" gate="G$1" x="226.06" y="154.94" smashed="yes" rot="MR0"/>
 <instance part="OFFSHEET9" gate="G$1" x="124.46" y="147.32" smashed="yes" rot="MR0"/>
-<instance part="OFFSHEET10" gate="G$1" x="53.34" y="58.42" smashed="yes" rot="MR0"/>
-<instance part="OFFSHEET12" gate="G$1" x="53.34" y="60.96" smashed="yes" rot="MR0"/>
+<instance part="OFFSHEET10" gate="G$1" x="58.42" y="58.42" smashed="yes" rot="MR0"/>
+<instance part="OFFSHEET12" gate="G$1" x="58.42" y="60.96" smashed="yes" rot="MR0"/>
 <instance part="OFFSHEET14" gate="G$1" x="137.16" y="93.98" smashed="yes" rot="MR0"/>
 <instance part="OFFSHEET17" gate="G$1" x="137.16" y="88.9" smashed="yes" rot="MR0"/>
@@
 <instance part="OFFSHEET27" gate="G$1" x="137.16" y="81.28" smashed="yes" rot="MR0"/>
 <instance part="OFFSHEET28" gate="G$1" x="137.16" y="78.74" smashed="yes" rot="MR0"/>
-<instance part="OFFSHEET34" gate="G$1" x="53.34" y="81.28" smashed="yes" rot="MR0"/>
-<instance part="OFFSHEET35" gate="G$1" x="53.34" y="76.2" smashed="yes" rot="MR0"/>
-<instance part="OFFSHEET40" gate="G$1" x="53.34" y="93.98" smashed="yes" rot="MR0"/>
-<instance part="OFFSHEET41" gate="G$1" x="53.34" y="91.44" smashed="yes" rot="MR0"/>
-<instance part="OFFSHEET42" gate="G$1" x="53.34" y="88.9" smashed="yes" rot="MR0"/>
+<instance part="OFFSHEET34" gate="G$1" x="58.42" y="81.28" smashed="yes" rot="MR0"/>
+<instance part="OFFSHEET35" gate="G$1" x="58.42" y="76.2" smashed="yes" rot="MR0"/>
+<instance part="OFFSHEET40" gate="G$1" x="58.42" y="93.98" smashed="yes" rot="MR0"/>
+<instance part="OFFSHEET41" gate="G$1" x="58.42" y="91.44" smashed="yes" rot="MR0"/>
+<instance part="OFFSHEET42" gate="G$1" x="58.42" y="88.9" smashed="yes" rot="MR0"/>
 <instance part="SW1" gate="G$1" x="198.12" y="50.8" smashed="yes">
 <attribute name="NAME" x="198.12" y="64.77" size="1.778" layer="95" align="center"/>
@@
 <instance part="SUPPLY32" gate="1" x="58.42" y="167.64" smashed="yes"/>
 <instance part="SUPPLY60" gate="1" x="38.1" y="124.46" smashed="yes"/>
-<instance part="OFFSHEET25" gate="G$1" x="53.34" y="83.82" smashed="yes" rot="MR0"/>
-<instance part="OFFSHEET11" gate="G$1" x="53.34" y="55.88" smashed="yes" rot="MR0"/>
-<instance part="OFFSHEET47" gate="G$1" x="53.34" y="66.04" smashed="yes" rot="MR0"/>
+<instance part="OFFSHEET25" gate="G$1" x="58.42" y="83.82" smashed="yes" rot="MR0"/>
+<instance part="OFFSHEET11" gate="G$1" x="58.42" y="55.88" smashed="yes" rot="MR0"/>
+<instance part="OFFSHEET47" gate="G$1" x="58.42" y="66.04" smashed="yes" rot="MR0"/>
 </instances>
 <busses>
@@
 <segment>
 <label x="35.56" y="71.12" size="1.778" layer="95"/>
-<wire x1="33.02" y1="71.12" x2="50.8" y2="71.12" width="0.1524" layer="91"/>
+<wire x1="33.02" y1="71.12" x2="55.88" y2="71.12" width="0.1524" layer="91"/>
 <pinref part="U1" gate="A" pin="PA9"/>
 </segment>
@@
 <segment>
 <label x="35.56" y="68.58" size="1.778" layer="95"/>
-<wire x1="33.02" y1="68.58" x2="50.8" y2="68.58" width="0.1524" layer="91"/>
+<wire x1="33.02" y1="68.58" x2="55.88" y2="68.58" width="0.1524" layer="91"/>
 <pinref part="U1" gate="A" pin="PA10"/>
 </segment>
@@
 <net name="I_ADJ" class="0">
 <segment>
-<wire x1="33.02" y1="83.82" x2="50.8" y2="83.82" width="0.1524" layer="91"/>
+<wire x1="33.02" y1="83.82" x2="55.88" y2="83.82" width="0.1524" layer="91"/>
 <label x="35.306" y="84.328" size="1.778" layer="95"/>
 <pinref part="U1" gate="A" pin="PA4"/>
@@
 </segment>
 <segment>
-<wire x1="33.02" y1="58.42" x2="50.8" y2="58.42" width="0.1524" layer="91"/>
+<wire x1="33.02" y1="58.42" x2="55.88" y2="58.42" width="0.1524" layer="91"/>
 <label x="35.56" y="58.42" size="1.778" layer="95"/>
 <pinref part="U1" gate="A" pin="PA14"/>
@@
 </segment>
 <segment>
-<wire x1="33.02" y1="60.96" x2="50.8" y2="60.96" width="0.1524" layer="91"/>
+<wire x1="33.02" y1="60.96" x2="55.88" y2="60.96" width="0.1524" layer="91"/>
 <label x="35.56" y="60.96" size="1.778" layer="95"/>
 <pinref part="U1" gate="A" pin="PA13"/>
@@
 <net name="JTAG_TDI" class="0">
 <segment>
-<wire x1="33.02" y1="55.88" x2="50.8" y2="55.88" width="0.1524" layer="91"/>
+<wire x1="33.02" y1="55.88" x2="55.88" y2="55.88" width="0.1524" layer="91"/>
 <label x="35.56" y="55.88" size="1.778" layer="95"/>
 <pinref part="U1" gate="A" pin="PA15"/>
@@
 <net name="SPI_SCK" class="0">
 <segment>
-<wire x1="33.02" y1="81.28" x2="50.8" y2="81.28" width="0.1524" layer="91"/>
+<wire x1="33.02" y1="81.28" x2="55.88" y2="81.28" width="0.1524" layer="91"/>
 <label x="35.56" y="81.28" size="1.778" layer="95"/>
 <pinref part="U1" gate="A" pin="PA5"/>
@@
 <net name="SPI_MOSI" class="0">
 <segment>
-<wire x1="33.02" y1="76.2" x2="50.8" y2="76.2" width="0.1524" layer="91"/>
+<wire x1="33.02" y1="76.2" x2="55.88" y2="76.2" width="0.1524" layer="91"/>
 <label x="35.56" y="76.2" size="1.778" layer="95"/>
 <pinref part="U1" gate="A" pin="PA7"/>
@@
 <net name="A0_LCD" class="0">
 <segment>
-<wire x1="33.02" y1="93.98" x2="50.8" y2="93.98" width="0.1524" layer="91"/>
+<wire x1="33.02" y1="93.98" x2="55.88" y2="93.98" width="0.1524" layer="91"/>
 <label x="35.56" y="93.98" size="1.778" layer="95"/>
 <pinref part="U1" gate="A" pin="PA0"/>
@@
 <net name="RST_LCD" class="0">
 <segment>
-<wire x1="33.02" y1="91.44" x2="50.8" y2="91.44" width="0.1524" layer="91"/>
+<wire x1="33.02" y1="91.44" x2="55.88" y2="91.44" width="0.1524" layer="91"/>
 <label x="35.56" y="91.44" size="1.778" layer="95"/>
 <pinref part="U1" gate="A" pin="PA1"/>
@@
 <net name="CS_LCD" class="0">
 <segment>
-<wire x1="33.02" y1="88.9" x2="50.8" y2="88.9" width="0.1524" layer="91"/>
+<wire x1="33.02" y1="88.9" x2="55.88" y2="88.9" width="0.1524" layer="91"/>
 <label x="35.56" y="88.9" size="1.778" layer="95"/>
 <pinref part="U1" gate="A" pin="PA2"/>
@@
 <net name="FAN_SENSE" class="0">
 <segment>
-<wire x1="33.02" y1="66.04" x2="50.8" y2="66.04" width="0.1524" layer="91"/>
+<wire x1="38.1" y1="66.04" x2="55.88" y2="66.04" width="0.1524" layer="91"/>
 <label x="35.56" y="66.04" size="1.778" layer="95"/>
 <label x="35.56" y="66.04" size="1.778" layer="95"/>
 </segment>
 </net>
+<net name="FAN_CONTROL" class="0">
+<segment>
+<pinref part="U1" gate="A" pin="PA6"/>
+<wire x1="33.02" y1="78.74" x2="55.88" y2="78.74" width="0.1524" layer="91"/>
+<label x="35.56" y="78.74" size="1.778" layer="95"/>
+</segment>
+</net>

Commit message: Update ElectronicLoad.sch
Connections:
- net FAN_DC renamed 12.0V
Changed lines of the file:
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@@
 <part name="OFFSHEET49" library="CougsInSpace-Aesthetics" deviceset="OFF_SHEET-IN" device=""/>
 <part name="OFFSHEET50" library="CougsInSpace-Aesthetics" deviceset="OFF_SHEET-IN" device=""/>
-<part name="OFFSHEET51" library="CougsInSpace-Aesthetics" deviceset="OFF_SHEET-IN" device=""/>
+<part name="SUPPLY67" library="CougsInSpace-PowerSymbols" deviceset="12.0V" device=""/>
 </parts>
 <sheets>
@@
 <text x="106.68" y="157.48" size="1.778" layer="95" align="center-left"> &lt;2C2</text>
 <text x="106.68" y="154.94" size="1.778" layer="95" align="center-left"> &lt;2C2</text>
-<text x="106.68" y="160.02" size="1.778" layer="95" align="center-left"> &lt;2C2</text>
 </plain>
 <instances>
@@
 <instance part="OFFSHEET49" gate="G$1" x="104.14" y="157.48" smashed="yes" rot="MR0"/>
 <instance part="OFFSHEET50" gate="G$1" x="104.14" y="154.94" smashed="yes" rot="MR0"/>
-<instance part="OFFSHEET51" gate="G$1" x="104.14" y="160.02" smashed="yes" rot="MR0"/>
+<instance part="SUPPLY67" gate="G$1" x="109.22" y="162.56" smashed="yes">
+<attribute name="VALUE" x="109.22" y="166.116" size="1.27" layer="96" align="center"/>
+</instance>
 </instances>
 <busses>
@@
 </segment>
 </net>
-<net name="FAN_DC" class="0">
-<segment>
-<pinref part="J6" gate="G$1" pin="2"/>
-<wire x1="81.28" y1="160.02" x2="101.6" y2="160.02" width="0.1524" layer="91"/>
-<label x="83.82" y="160.02" size="1.778" layer="95"/>
-</segment>
-</net>
 <net name="FAN_GND" class="0">
 <segment>
@@
 </segment>
 </net>
+<net name="12.0V" class="0">
+<segment>
+<pinref part="J6" gate="G$1" pin="2"/>
+<wire x1="81.28" y1="160.02" x2="109.22" y2="160.02" width="0.1524" layer="91"/>
+<label x="83.82" y="160.02" size="1.778" layer="95"/>
+<pinref part="SUPPLY67" gate="G$1" pin="12.0V"/>
+<wire x1="109.22" y1="160.02" x2="109.22" y2="162.56" width="0.1524" layer="91"/>
+</segment>
+</net>

Commit message: Fixed it part (100,000,000)
Parts:
- added J7: (no value), CougsInSpace-Connectors:BARREL-2.1X5.5-R
- added R18: 0Ω <20mΩ, CougsInSpace-Resistors:RES-V-0-1608
Connections:
- removed net FAN_GND: J6.1
- new net PGND: J6.1, J7.SLEEVE, J7.SW, R18.1
- net 12.0V: now also J7.CENTER
- net CHASSIS: now also R18.2
Other:
- note added: "3A3>"
Changed lines of the file:
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@@
 <part name="OFFSHEET11" library="CougsInSpace-Aesthetics" deviceset="OFF_SHEET-OUT" device=""/>
 <part name="J6" library="CougsInSpace-Connectors" deviceset="1X04" device="THT2.54-1X04-LOCK"/>
-<part name="SUPPLY66" library="CougsInSpace-PowerSymbols" deviceset="DGND" device=""/>
 <part name="OFFSHEET47" library="CougsInSpace-Aesthetics" deviceset="OFF_SHEET-OUT" device=""/>
 <part name="OFFSHEET49" library="CougsInSpace-Aesthetics" deviceset="OFF_SHEET-IN" device=""/>
 <part name="OFFSHEET50" library="CougsInSpace-Aesthetics" deviceset="OFF_SHEET-IN" device=""/>
-<part name="SUPPLY67" library="CougsInSpace-PowerSymbols" deviceset="12.0V" device=""/>
+<part name="SUPPLY66" library="CougsInSpace-PowerSymbols" deviceset="12.0V" device=""/>
+<part name="SUPPLY67" library="CougsInSpace-PowerSymbols" deviceset="PGND" device=""/>
+<part name="OFFSHEET51" library="CougsInSpace-Aesthetics" deviceset="OFF_SHEET-OUT" device=""/>
+<part name="J7" library="CougsInSpace-Connectors" deviceset="BARREL" device="-2.1X5.5-R"/>
+<part name="SUPPLY68" library="CougsInSpace-PowerSymbols" deviceset="12.0V" device=""/>
+<part name="SUPPLY69" library="CougsInSpace-PowerSymbols" deviceset="PGND" device=""/>
+<part name="R18" library="CougsInSpace-Resistors" deviceset="RES-V" device="-1608" technology="-0" value="0Ω &lt;20mΩ"/>
+<part name="SUPPLY70" library="CougsInSpace-PowerSymbols" deviceset="PGND" device=""/>
 </parts>
 <sheets>
@@
 <wire x1="154.94" y1="53.34" x2="200.66" y2="53.34" width="0.1524" layer="94"/>
 <text x="177.8" y="60.96" size="3.81" layer="94" align="center">Heatsink &amp; Fan</text>
-<text x="199.39" y="54.61" size="1.778" layer="97" align="bottom-right">Page 2</text>
+<text x="199.39" y="54.61" size="1.778" layer="97" align="bottom-right">Page 3</text>
 <wire x1="177.8" y1="81.28" x2="177.8" y2="68.58" width="0.254" layer="97"/>
 <text x="178.054" y="74.93" size="1.778" layer="97" align="center-left">Thermal</text>
@@
 <text x="60.96" y="93.98" size="1.778" layer="95" align="center-left"> 3C5&gt;</text>
 <text x="60.96" y="91.44" size="1.778" layer="95" align="center-left"> 3C5&gt;</text>
-<text x="60.96" y="88.9" size="1.778" layer="95" align="center-left"> 3C5&gt;</text>
+<text x="60.96" y="88.9" size="1.778" layer="95" align="center-left"> 3A3&gt;</text>
 <text x="60.96" y="81.28" size="1.778" layer="95" align="center-left"> 3C5&gt;</text>
 <text x="60.96" y="76.2" size="1.778" layer="95" align="center-left"> 3C5&gt;</text>
@@
 <text x="83.82" y="163.83" size="1.778" layer="97" align="center">CAD Note: Decoupling</text>
 <text x="60.96" y="66.04" size="1.778" layer="95" align="center-left"> 3A2&gt;</text>
+<text x="60.96" y="78.74" size="1.778" layer="95" align="center-left"> 3C5&gt;</text>
 </plain>
 <instances>
@@
 <instance part="OFFSHEET11" gate="G$1" x="58.42" y="55.88" smashed="yes" rot="MR0"/>
 <instance part="OFFSHEET47" gate="G$1" x="58.42" y="66.04" smashed="yes" rot="MR0"/>
+<instance part="OFFSHEET51" gate="G$1" x="58.42" y="78.74" smashed="yes" rot="MR0"/>
+<instance part="J7" gate="G$1" x="157.48" y="162.56" smashed="yes">
+<attribute name="NAME" x="157.48" y="171.45" size="1.778" layer="95" align="center"/>
+<attribute name="VALUE" x="157.48" y="153.67" size="1.778" layer="96" align="center"/>
+<attribute name="SKU" x="157.48" y="151.638" size="1.778" layer="97" align="center"/>
+</instance>
+<instance part="SUPPLY68" gate="G$1" x="172.72" y="167.64" smashed="yes">
+<attribute name="VALUE" x="172.72" y="171.196" size="1.27" layer="96" align="center"/>
+</instance>
+<instance part="SUPPLY69" gate="G$1" x="172.72" y="152.4" smashed="yes"/>
 </instances>
 <busses>
@@
 <segment>
 <pinref part="J5" gate="G$1" pin="SWCLK"/>
-<wire x1="203.2" y1="160.02" x2="223.52" y2="160.02" width="0.1524" layer="91"/>
+<wire x1="203.2" y1="160.02" x2="259.08" y2="144.78" width="0.1524" layer="91"/>
 <label x="208.28" y="160.02" size="1.778" layer="95"/>
 </segment>
@@
 <wire x1="33.02" y1="78.74" x2="55.88" y2="78.74" width="0.1524" layer="91"/>
 <label x="35.56" y="78.74" size="1.778" layer="95"/>
+</segment>
+</net>
+<net name="PGND" class="0">
+<segment>
+<pinref part="J7" gate="G$1" pin="SLEEVE"/>
+<wire x1="167.64" y1="157.48" x2="172.72" y2="157.48" width="0.1524" layer="91"/>
+<pinref part="SUPPLY69" gate="G$1" pin="PGND"/>
+<wire x1="172.72" y1="157.48" x2="172.72" y2="154.94" width="0.1524" layer="91"/>
+<pinref part="J7" gate="G$1" pin="SW"/>
+<wire x1="167.64" y1="160.02" x2="172.72" y2="160.02" width="0.1524" layer="91"/>
+<wire x1="172.72" y1="160.02" x2="172.72" y2="157.48" width="0.1524" layer="91"/>
+<junction x="172.72" y="157.48"/>
+</segment>
+</net>
+<net name="12.0V" class="0">
+<segment>
+<pinref part="SUPPLY68" gate="G$1" pin="12.0V"/>
+<wire x1="172.72" y1="167.64" x2="172.72" y2="165.1" width="0.1524" layer="91"/>
+<pinref part="J7" gate="G$1" pin="CENTER"/>
+<wire x1="172.72" y1="165.1" x2="167.64" y2="165.1" width="0.1524" layer="91"/>
 </segment>
 </net>
@@
 </instance>
 <instance part="OFFSHEET16" gate="G$1" x="83.82" y="55.88" smashed="yes" rot="MR0"/>
-<instance part="OFFSHEET24" gate="G$1" x="106.68" y="132.08" smashed="yes" rot="MR0"/>
+<instance part="OFFSHEET24" gate="G$1" x="210.82" y="48.26" smashed="yes" rot="MR0"/>
 <instance part="J2" gate="G$1" x="144.78" y="142.24" smashed="yes">
 <attribute name="VALUE" x="145.415" y="138.43" size="1.778" layer="96" align="center"/>
@@
 <attribute name="PACKAGE" x="74.295" y="147.066" size="1.778" layer="97" align="center"/>
 </instance>
-<instance part="SUPPLY66" gate="1" x="104.14" y="162.56" smashed="yes" rot="R90"/>
 <instance part="OFFSHEET49" gate="G$1" x="104.14" y="157.48" smashed="yes" rot="MR0"/>
 <instance part="OFFSHEET50" gate="G$1" x="104.14" y="154.94" smashed="yes" rot="MR0"/>
-<instance part="SUPPLY67" gate="G$1" x="109.22" y="162.56" smashed="yes">
-<attribute name="VALUE" x="109.22" y="166.116" size="1.27" layer="96" align="center"/>
-</instance>
+<instance part="SUPPLY66" gate="G$1" x="96.52" y="162.56" smashed="yes">
+<attribute name="VALUE" x="96.52" y="166.116" size="1.27" layer="96" align="center"/>
+</instance>
+<instance part="SUPPLY67" gate="G$1" x="91.44" y="162.56" smashed="yes" rot="R90"/>
 </instances>
 <busses>
@@
 </segment>
 </net>
-<net name="FAN_GND" class="0">
+<net name="PGND" class="0">
 <segment>
 <pinref part="J6" gate="G$1" pin="1"/>
-<pinref part="SUPPLY66" gate="1" pin="DGND"/>
-<wire x1="101.6" y1="162.56" x2="81.28" y2="162.56" width="0.1524" layer="91"/>
-<label x="83.82" y="162.56" size="1.778" layer="95"/>
+<pinref part="SUPPLY67" gate="G$1" pin="PGND"/>
+<wire x1="88.9" y1="162.56" x2="81.28" y2="162.56" width="0.1524" layer="91"/>
 </segment>
 </net>
@@
 <segment>
 <pinref part="J6" gate="G$1" pin="2"/>
-<wire x1="81.28" y1="160.02" x2="109.22" y2="160.02" width="0.1524" layer="91"/>
-<label x="83.82" y="160.02" size="1.778" layer="95"/>
-<pinref part="SUPPLY67" gate="G$1" pin="12.0V"/>
-<wire x1="109.22" y1="160.02" x2="109.22" y2="162.56" width="0.1524" layer="91"/>
+<wire x1="81.28" y1="160.02" x2="96.52" y2="160.02" width="0.1524" layer="91"/>
+<pinref part="SUPPLY66" gate="G$1" pin="12.0V"/>
+<wire x1="96.52" y1="160.02" x2="96.52" y2="162.56" width="0.1524" layer="91"/>
 </segment>
 </net>
@@
 <attribute name="SKU" x="21.59" y="27.432" size="1.27" layer="97" rot="MR0" align="center-left"/>
 </instance>
+<instance part="R18" gate="G$1" x="40.64" y="25.4" smashed="yes" rot="MR0">
+<attribute name="NAME" x="39.37" y="30.48" size="1.27" layer="95" rot="MR0" align="center-left"/>
+<attribute name="VALUE" x="39.37" y="28.956" size="1.27" layer="96" rot="MR0" align="center-left"/>
+<attribute name="PACKAGE" x="39.37" y="25.908" size="1.27" layer="97" rot="MR0" align="center-left"/>
+<attribute name="POWER" x="39.37" y="24.384" size="1.27" layer="97" rot="MR0" align="center-left"/>
+<attribute name="TEMP" x="39.37" y="22.86" size="1.27" layer="97" rot="MR0" align="center-left"/>
+<attribute name="SKU" x="39.37" y="27.432" size="1.27" layer="97" rot="MR0" align="center-left"/>
+</instance>
+<instance part="SUPPLY70" gate="G$1" x="40.64" y="15.24" smashed="yes"/>
 </instances>
 <busses>
@@
 <pinref part="R17" gate="G$1" pin="2"/>
 <wire x1="22.86" y1="33.02" x2="22.86" y2="30.48" width="0.1524" layer="91"/>
+<pinref part="R18" gate="G$1" pin="2"/>
+<wire x1="40.64" y1="30.48" x2="40.64" y2="33.02" width="0.1524" layer="91"/>
+<wire x1="40.64" y1="33.02" x2="27.94" y2="33.02" width="0.1524" layer="91"/>
+<junction x="27.94" y="33.02"/>
 </segment>
 </net>
@@
 </segment>
 </net>
+<net name="PGND" class="0">
+<segment>
+<pinref part="R18" gate="G$1" pin="1"/>
+<pinref part="SUPPLY70" gate="G$1" pin="PGND"/>
+<wire x1="40.64" y1="22.86" x2="40.64" y2="17.78" width="0.1524" layer="91"/>
+</segment>
+</net>
