File: Subsystems/Electronics/Testing/ElectronicLoad/ElectricalDesign/ElectronicLoad.brd (EAGLE design)
At the start: 104 x 130 mm, 85 parts, among them J1 USB, J2 Load, J3 Alternate Current Sense, J4 Voltage Sense, J5 SWD, J6 FAN, J7 12 V Input, Q1 IRFP4368PBF, Q2 SiRA20DP, Q3 SiRA20DP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

Commit message: Update ElectronicLoad.brd
Parts:
- moved R13 19.2 mm to (42.0, -7.00), turned to 0 degrees
- moved R15 17.0 mm to (39.0, -5.00), turned to 180 degrees
- moved C9 12.1 mm to (33.0, -15.0), turned to 180 degrees
- moved R7 11.0 mm to (39.0, -7.00), turned to 0 degrees
- moved R4 10.8 mm to (45.0, -5.00), turned to 0 degrees
- moved C16 10.3 mm to (-40.0, -10.0), turned to 0 degrees
- moved C7 10.3 mm to (33.0, -13.0), turned to 180 degrees
- moved C14 9.49 mm to (-36.0, -10.0), turned to 0 degrees
- moved C20 9.06 mm to (-32.0, -10.0), turned to 0 degrees
- moved C22 9.06 mm to (-28.0, -10.0), turned to 0 degrees
- moved B1 8.60 mm to (-44.0, -36.0)
- moved C6 8.60 mm to (33.0, -11.0), turned to 180 degrees
- moved RN1 8.25 mm to (-16.0, -51.0)
- moved C17 8.06 mm to (-44.0, -12.0), turned to 180 degrees
- moved DS1 8.06 mm to (-18.0, -24.0), turned to 180 degrees
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
Commit message: Layout_placement
Parts:
- moved J1 89.5 mm to (-43.0, -12.0), turned to 270 degrees
- moved J6 81.4 mm to (24.0, -8.00)
- moved R2 75.7 mm to (38.0, -58.0), flipped to the bottom
- moved U1 71.6 mm to (-28.0, 46.0)
- moved J5 40.5 mm to (-33.0, -32.0), flipped to the bottom, turned to 90 degrees
- moved R6 26.2 mm to (15.0, 3.00)
- moved C17 20.6 mm to (-25.0, -20.0)
- moved C15 16.2 mm to (-25.0, -18.0)
- moved C16 14.4 mm to (-28.0, -18.0)
- moved U3 13.4 mm to (26.0, -22.0)
- moved R19 13.2 mm to (-31.0, -8.00)
- moved C26 13.0 mm to (-31.0, -4.00)
- moved C27 13.0 mm to (-31.0, -6.00)
- moved C11 12.0 mm to (-28.0, -4.00)
- moved C25 12.0 mm to (-28.0, -6.00)
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Routing:
- net DGND: track 0.00 -> 32.2 mm
- net CHASSIS: track 0.00 -> 25.5 mm
- net 3.1V: track 0.00 -> 22.9 mm
- net PGND: track 0.00 -> 2.00 mm

Commit message: FIxes_to_layout
Parts:
- moved U4 41.1 mm to (21.0, -27.0), turned to 0 degrees
- moved U2 26.6 mm to (15.0, -22.0)
- moved Y1 22.0 mm to (3.00, -24.0)
- moved R11 17.5 mm to (13.0, -27.0), turned to 0 degrees
- moved R1 15.6 mm to (9.00, -7.00), turned to 270 degrees
- moved R5 15.0 mm to (9.00, -10.0), turned to 270 degrees
- moved R8 15.0 mm to (9.00, -18.0)
- moved R9 13.6 mm to (7.00, -18.0)
- moved R22 13.0 mm to (8.00, -21.0), turned to 0 degrees
- moved C19 9.22 mm to (-34.0, -20.0)
- moved U6 7.21 mm to (-13.0, -15.0)
- moved R17 4.00 mm to (-24.0, -12.0), turned to 270 degrees
- moved R2 3.16 mm to (39.0, -55.0)
- moved C24 3.00 mm to (-25.0, -9.00), turned to 0 degrees
- moved C1 2.24 mm to (-25.0, -7.00)
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Routing:
- net DGND: track 32.2 -> 1.00 mm
- net CHASSIS: track 25.5 -> 0.00 mm
- net 3.1V: track 22.9 -> 0.79 mm
- net PGND: track 2.00 -> 0.00 mm

Commit message: Updated board layout
Parts:
- moved R6 82.6 mm to (-66.0, -13.0)
- moved R20 80.7 mm to (-83.0, 4.00), turned to 180 degrees
- moved Y1 77.8 mm to (-74.0, -13.0), turned to 180 degrees
- moved R4 76.2 mm to (-31.0, -11.0)
- moved R5 74.1 mm to (-65.0, -7.00), turned to 180 degrees
- moved R1 74.0 mm to (-65.0, -9.00), turned to 0 degrees
- moved R22 73.1 mm to (-65.0, -17.0)
- moved R10 70.5 mm to (-85.0, 0.00), turned to 90 degrees
- moved DS1 68.0 mm to (-83.0, -4.00), turned to 0 degrees
- moved C4 67.0 mm to (-34.0, -9.00), turned to 0 degrees
- moved R3 64.5 mm to (-31.0, -13.0)
- moved C5 64.0 mm to (-31.0, -9.00)
- moved C10 63.3 mm to (-87.0, -18.0)
- moved C11 63.3 mm to (-90.0, -18.0)
- moved C25 63.3 mm to (-90.0, -20.0), turned to 0 degrees
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Routing:
- net 3.1V: track 0.79 -> 0.00 mm
- net DGND: track 1.00 -> 0.50 mm

Commit message: Fixed-IC-placement
Parts:
- moved C26 127.5 mm to (37.0, -26.0)
- moved C25 116.1 mm to (26.0, -15.0)
- moved C27 75.4 mm to (-23.0, -43.0)
- moved C24 69.0 mm to (-12.0, -18.0)
Changed lines of the file:
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@@
 <attribute name="VOLTAGE" value="100V" x="-166.44" y="-23.24" size="1.778" layer="27" rot="R270" display="off"/>
 </element>
-<element name="C24" library="CougsInSpace-Capacitors" package="1608" value="100nF 10%" x="-81" y="-20" smashed="yes">
-<attribute name="NAME" x="-81" y="-21.6" size="0.8" layer="25" font="vector" ratio="15" align="center"/>
-<attribute name="PACKAGE" value="1608" x="-61.95" y="-111.44" size="1.778" layer="27" display="off"/>
-<attribute name="SKU" value="11-104A" x="-61.95" y="-111.44" size="1.778" layer="27" display="off"/>
-<attribute name="TEMP" value="X7R" x="-61.95" y="-111.44" size="1.778" layer="27" display="off"/>
-<attribute name="VOLTAGE" value="50V" x="-61.95" y="-111.44" size="1.778" layer="27" display="off"/>
-</element>
-<element name="C25" library="CougsInSpace-Capacitors" package="1608" value="100nF 10%" x="-90" y="-20" smashed="yes">
-<attribute name="NAME" x="-90" y="-21.6" size="0.8" layer="25" font="vector" ratio="15" align="center"/>
-<attribute name="PACKAGE" value="1608" x="-67.14" y="-111.44" size="1.778" layer="27" display="off"/>
-<attribute name="SKU" value="11-104A" x="-67.14" y="-111.44" size="1.778" layer="27" display="off"/>
-<attribute name="TEMP" value="X7R" x="-67.14" y="-111.44" size="1.778" layer="27" display="off"/>
-<attribute name="VOLTAGE" value="50V" x="-67.14" y="-111.44" size="1.778" layer="27" display="off"/>
-</element>
-<element name="C26" library="CougsInSpace-Capacitors" package="1608" value="100nF 10%" x="-90" y="-15" smashed="yes" rot="R180">
-<attribute name="NAME" x="-90" y="-13.4" size="0.8" layer="25" font="vector" ratio="15" rot="R180" align="center"/>
-<attribute name="PACKAGE" value="1608" x="-116.67" y="76.44" size="1.778" layer="27" rot="R180" display="off"/>
-<attribute name="SKU" value="11-104A" x="-116.67" y="76.44" size="1.778" layer="27" rot="R180" display="off"/>
-<attribute name="TEMP" value="X7R" x="-116.67" y="76.44" size="1.778" layer="27" rot="R180" display="off"/>
-<attribute name="VOLTAGE" value="50V" x="-116.67" y="76.44" size="1.778" layer="27" rot="R180" display="off"/>
-</element>
-<element name="C27" library="CougsInSpace-Capacitors" package="1608" value="100nF 10%" x="-93" y="-15" smashed="yes" rot="R180">
-<attribute name="NAME" x="-93" y="-13.4" size="0.8" layer="25" font="vector" ratio="15" rot="R180" align="center"/>
-<attribute name="PACKAGE" value="1608" x="-123.48" y="76.44" size="1.778" layer="27" rot="R180" display="off"/>
-<attribute name="SKU" value="11-104A" x="-123.48" y="76.44" size="1.778" layer="27" rot="R180" display="off"/>
-<attribute name="TEMP" value="X7R" x="-123.48" y="76.44" size="1.778" layer="27" rot="R180" display="off"/>
-<attribute name="VOLTAGE" value="50V" x="-123.48" y="76.44" size="1.778" layer="27" rot="R180" display="off"/>
+<element name="C24" library="CougsInSpace-Capacitors" package="1608" value="100nF 10%" x="-12" y="-18" smashed="yes">
+<attribute name="NAME" x="-12" y="-19.6" size="0.8" layer="25" font="vector" ratio="15" align="center"/>
+<attribute name="PACKAGE" value="1608" x="7.05" y="-109.44" size="1.778" layer="27" display="off"/>
+<attribute name="SKU" value="11-104A" x="7.05" y="-109.44" size="1.778" layer="27" display="off"/>
+<attribute name="TEMP" value="X7R" x="7.05" y="-109.44" size="1.778" layer="27" display="off"/>
+<attribute name="VOLTAGE" value="50V" x="7.05" y="-109.44" size="1.778" layer="27" display="off"/>
+</element>
+<element name="C25" library="CougsInSpace-Capacitors" package="1608" value="100nF 10%" x="26" y="-15" smashed="yes">
+<attribute name="NAME" x="26" y="-16.6" size="0.8" layer="25" font="vector" ratio="15" align="center"/>
+<attribute name="PACKAGE" value="1608" x="48.86" y="-106.44" size="1.778" layer="27" display="off"/>
+<attribute name="SKU" value="11-104A" x="48.86" y="-106.44" size="1.778" layer="27" display="off"/>
+<attribute name="TEMP" value="X7R" x="48.86" y="-106.44" size="1.778" layer="27" display="off"/>
+<attribute name="VOLTAGE" value="50V" x="48.86" y="-106.44" size="1.778" layer="27" display="off"/>
+</element>
+<element name="C26" library="CougsInSpace-Capacitors" package="1608" value="100nF 10%" x="37" y="-26" smashed="yes" rot="R180">
+<attribute name="NAME" x="37" y="-24.4" size="0.8" layer="25" font="vector" ratio="15" rot="R180" align="center"/>
+<attribute name="PACKAGE" value="1608" x="10.33" y="65.44" size="1.778" layer="27" rot="R180" display="off"/>
+<attribute name="SKU" value="11-104A" x="10.33" y="65.44" size="1.778" layer="27" rot="R180" display="off"/>
+<attribute name="TEMP" value="X7R" x="10.33" y="65.44" size="1.778" layer="27" rot="R180" display="off"/>
+<attribute name="VOLTAGE" value="50V" x="10.33" y="65.44" size="1.778" layer="27" rot="R180" display="off"/>
+</element>
+<element name="C27" library="CougsInSpace-Capacitors" package="1608" value="100nF 10%" x="-23" y="-43" smashed="yes" rot="R180">
+<attribute name="NAME" x="-23" y="-41.4" size="0.8" layer="25" font="vector" ratio="15" rot="R180" align="center"/>
+<attribute name="PACKAGE" value="1608" x="-53.48" y="48.44" size="1.778" layer="27" rot="R180" display="off"/>
+<attribute name="SKU" value="11-104A" x="-53.48" y="48.44" size="1.778" layer="27" rot="R180" display="off"/>
+<attribute name="TEMP" value="X7R" x="-53.48" y="48.44" size="1.778" layer="27" rot="R180" display="off"/>
+<attribute name="VOLTAGE" value="50V" x="-53.48" y="48.44" size="1.778" layer="27" rot="R180" display="off"/>
 </element>
 <element name="C28" library="CougsInSpace-Capacitors" package="1608" value="1µF 10%" x="71" y="-23" smashed="yes">
@@
 <wire x1="-73" y1="-8.75" x2="-75" y2="-8.75" width="0" layer="19" extent="1-1"/>
 <wire x1="-80.25" y1="-18" x2="-75.85" y2="-11.9" width="0" layer="19" extent="1-1"/>
-<wire x1="-80.25" y1="-20" x2="-80.25" y2="-18" width="0" layer="19" extent="1-1"/>
+<wire x1="-11.25" y1="-18" x2="-80.25" y2="-18" width="0" layer="19" extent="1-1"/>
 <wire x1="-84.75" y1="-18" x2="-80.25" y2="-18" width="0" layer="19" extent="1-1"/>
 <wire x1="-86.25" y1="-18" x2="-84.75" y2="-18" width="0" layer="19" extent="1-1"/>
 <wire x1="-89.25" y1="-18" x2="-86.25" y2="-18" width="0" layer="19" extent="1-1"/>
-<wire x1="-89.25" y1="-20" x2="-89.25" y2="-18.5" width="0" layer="19" extent="1-1"/>
-<wire x1="-90.75" y1="-15" x2="-89.25" y2="-18" width="0" layer="19" extent="1-1"/>
-<wire x1="-93.75" y1="-15" x2="-90.75" y2="-15" width="0" layer="19" extent="1-1"/>
+<wire x1="26.75" y1="-15" x2="-89.25" y2="-18.5" width="0" layer="19" extent="1-1"/>
+<wire x1="36.25" y1="-26" x2="-89.25" y2="-18" width="0" layer="19" extent="1-1"/>
+<wire x1="-23.75" y1="-43" x2="36.25" y2="-26" width="0" layer="19" extent="1-1"/>
 <wire x1="-78.75" y1="-0.25" x2="-75" y2="-8.75" width="0" layer="19" extent="1-1"/>
 <wire x1="-85" y1="-0.75" x2="-78.75" y2="-0.25" width="0" layer="19" extent="1-1"/>
@@
 <contactref element="C8" pad="A"/>
 <contactref element="TP6" pad="1"/>
-<wire x1="-21" y1="-8" x2="-90.75" y2="-20" width="0" layer="19" extent="1-1"/>
+<wire x1="-21" y1="-8" x2="25.25" y2="-15" width="0" layer="19" extent="1-1"/>
 <wire x1="14.05" y1="-20.69" x2="-21" y2="-8" width="0" layer="19" extent="1-1"/>
 <wire x1="-17.6" y1="-14.35" x2="14.05" y2="-20.69" width="0" layer="19" extent="1-1"/>
@@
 <contactref element="C3" pad="1"/>
 <wire x1="-87.75" y1="-18" x2="-90.75" y2="-18" width="0" layer="19" extent="1-1"/>
-<wire x1="-92.25" y1="-15" x2="-90.75" y2="-18" width="0" layer="19" extent="1-1"/>
-<wire x1="-89.25" y1="-15" x2="-92.25" y2="-15" width="0" layer="19" extent="1-1"/>
+<wire x1="-22.25" y1="-43" x2="-90.75" y2="-18" width="0" layer="19" extent="1-1"/>
+<wire x1="37.75" y1="-26" x2="-22.25" y2="-43" width="0" layer="19" extent="1-1"/>
 <wire x1="-83.25" y1="-18" x2="-87.75" y2="-18" width="0" layer="19" extent="1-1"/>
 <wire x1="-81.75" y1="-18" x2="-83.25" y2="-18" width="0" layer="19" extent="1-1"/>
-<wire x1="-81.75" y1="-20" x2="-81.75" y2="-18" width="0" layer="19" extent="1-1"/>
+<wire x1="-12.75" y1="-18" x2="-81.75" y2="-18" width="0" layer="19" extent="1-1"/>
 <wire x1="-76.75" y1="-2.75" x2="-81.75" y2="-18" width="0" layer="19" extent="1-1"/>
 <wire x1="-78.75" y1="-0.75" x2="-76.75" y2="-2.75" width="0" layer="19" extent="1-1"/>
@@
 <wire x1="-67.25" y1="6.75" x2="-76.75" y2="8.75" width="0" layer="19" extent="1-1"/>
 <wire x1="-67.25" y1="0.25" x2="-67.25" y2="6.75" width="0" layer="19" extent="1-1"/>
-<wire x1="-54.25" y1="-26" x2="-81.75" y2="-20" width="0" layer="19" extent="1-1"/>
+<wire x1="-54.25" y1="-26" x2="-12.75" y2="-18" width="0" layer="19" extent="1-1"/>
 <wire x1="-49" y1="-46.5" x2="-54.25" y2="-26" width="0" layer="19" extent="1-1"/>
 <wire x1="-23.2" y1="-46.7" x2="-49" y2="-46.5" width="0" layer="19" extent="1-1"/>

Commit message: modified-layout
Parts:
- moved C1 107.7 mm to (26.2, -28.0)
- moved C10 107.7 mm to (20.2, -28.0)
- moved C11 107.7 mm to (17.2, -28.0)
- moved C2 107.7 mm to (23.2, -28.0)
- moved R1 101.2 mm to (35.5, -20.5), turned to 90 degrees
- moved R6 98.5 mm to (32.2, -19.5), turned to 0 degrees
- moved R22 93.8 mm to (28.8, -20.8)
- moved R5 90.5 mm to (24.8, -19.0)
- moved R20 87.2 mm to (2.75, -12.0)
- moved DS1 87.0 mm to (2.50, -20.2)
- moved U1 87.0 mm to (12.5, -13.0)
- moved R10 86.7 mm to (-0.50, -19.5)
- moved C18 85.6 mm to (11.2, -23.0)
- moved Y1 85.5 mm to (10.2, -27.5)
- moved C23 85.1 mm to (8.75, -23.0)
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
Commit message: worked on layout
Parts:
- moved C24 6.25 mm to (26.2, -23.8)
- moved C25 4.56 mm to (23.8, -14.2)
- moved C28 2.26 mm to (40.2, -16.5)
- moved C29 2.26 mm to (40.2, -14.5)
- moved R5 2.15 mm to (26.0, -17.2)
- moved U5 1.77 mm to (39.8, -10.5)
- moved U6 1.68 mm to (30.8, -13.2)
- moved R9 1.27 mm to (19.0, -23.8)
- moved R8 1.25 mm to (21.8, -23.8)
- moved C21 0.75 mm to (-21.8, -41.8)
- moved C18 0.25 mm to (11.2, -23.2)
- moved R19 0.25 mm to (-21.8, -44.2)
Routing:
- net CHASSIS: track 0.00 -> 517.8 mm, vias 0 -> 4
- net DGND: track 0.50 -> 382.7 mm, vias 0 -> 35
- net 3.1V: track 0.00 -> 250.8 mm, vias 0 -> 20
- net LOAD_INPUT+: track 0.00 -> 146.8 mm, vias 0 -> 4
- net FEEDBACK: track 0.00 -> 145.9 mm, vias 0 -> 6
- net PGND: track 0.00 -> 125.4 mm, vias 0 -> 6
- net SPI_SCK: track 0.00 -> 120.0 mm, vias 0 -> 8
- net 5.0V: track 0.00 -> 118.0 mm, vias 0 -> 12
- net SPI_MOSI: track 0.00 -> 108.9 mm, vias 0 -> 6
- net !LCD_CS: track 0.00 -> 105.1 mm, vias 0 -> 4
- net LCD_A0: track 0.00 -> 104.2 mm, vias 0 -> 6
- net !LCD_RST: track 0.00 -> 103.8 mm, vias 0 -> 4
- net FET_GATE: track 0.00 -> 89.9 mm, vias 0 -> 11
- net SHUNT_LOW: track 0.00 -> 86.7 mm, vias 0 -> 2
- net ENC_SW: track 0.00 -> 78.8 mm, vias 0 -> 5
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
Commit message: Board Layout finished
Parts:
- moved C23 2.15 mm to (7.50, -21.2)
- moved Y1 1.25 mm to (10.2, -28.8)
- moved J4 0.79 mm to (18.8, -35.8)
- moved R4 0.79 mm to (-15.1, -8.10)
- moved R13 0.75 mm to (-15.9, -5.60)
- moved C14 0.56 mm to (-22.2, -48.8)
- moved C16 0.56 mm to (-22.0, -53.0)
- moved C15 0.50 mm to (-21.8, -51.0)
- moved C18 0.50 mm to (11.2, -23.8)
- moved R1 0.25 mm to (35.8, -20.5)
- moved R20 0.25 mm to (2.75, -11.8)
- moved R3 0.25 mm to (-14.8, -11.5)
Routing:
- net SHUNT_MID: track 42.5 -> 111.8 mm, vias 2 -> 3
- net DGND: track 382.7 -> 415.5 mm
- net 3.1V: track 250.8 -> 281.7 mm, vias 20 -> 22
- net SWO: track 38.8 -> 69.1 mm, vias 1 -> 4
- net ENC_B: track 53.0 -> 66.9 mm, vias 3 -> 4
- net CHASSIS: track 517.8 -> 531.6 mm
- net AVDD: track 48.2 -> 55.8 mm, vias 0 -> 6
- net V_ALT: track 41.2 -> 47.2 mm, vias 0 -> 2
- net FEEDBACK: track 145.9 -> 140.7 mm
- net OSC_OUT: track 9.76 -> 13.9 mm, vias 4 -> 5
- net LOAD_INPUT-: track 30.0 -> 34.0 mm
- net SHUNT_LOW: track 86.7 -> 90.2 mm
- net OSC_IN: track 12.4 -> 14.7 mm
- net FET_GATE: track 89.9 -> 91.7 mm
- net I_LOAD: track 59.3 -> 58.0 mm
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