File: Subsystems/Electronics/Testing/ElectronicLoad/ElectricalDesign/ElectronicLoad.brd (EAGLE design)
At the start: 104 x 130 mm, 85 parts, among them J1 USB, J2 Load, J3 Alternate Current Sense, J4 Voltage Sense, J5 SWD, J6 FAN, J7 12 V Input, Q1 IRFP4368PBF, Q2 SiRA20DP, Q3 SiRA20DP, Q4 IRFP4368PBF, SW1 Nice Knob, SW2 Nice Button, U1 STM32L476RGT, U2 AD8515, U3 FT230XQ, U4 INA199C1, U5 LP5907MFX-3.1, U6 INA199C1, Y1 8MHz ±10ppm

Commit message: Finished board layout
Parts:
- added C30, C31: 1µF 10%, CougsInSpace-Capacitors:1608
- added D1, D2: LTC4411, CougsInSpace-DiscreteSemi:SOT23-5
- added R25: 10kΩ 0.1%, CougsInSpace-Resistors:1608
- added R26: 30kΩ 1%, CougsInSpace-Resistors:1608
- added U7: TPS73250, CougsInSpace-IC-Power:SOT23-5
- moved Q3 66.9 mm to (34.0, -22.6), turned to 90 degrees
- moved Q2 58.1 mm to (26.9, -22.1)
- moved U4 26.0 mm to (15.2, -12.8)
- moved C28 26.0 mm to (14.8, -21.9)
- moved C29 25.9 mm to (14.9, -9.40)
- moved U5 25.7 mm to (15.2, -17.9)
- moved J6 23.3 mm to (47.3, -9.15), turned to 270 degrees
- moved C26 21.5 mm to (17.8, -24.8)
- moved B1 21.3 mm to (-27.8, -43.8), turned to 90 degrees
- moved C9 20.8 mm to (-34.1, -10.7), turned to 180 degrees
- moved C12 20.3 mm to (-10.9, -21.6)
- moved U3 20.3 mm to (-30.1, -11.9)
- moved R4 19.8 mm to (-34.1, -13.5), turned to 0 degrees
- moved C4 19.2 mm to (-36.5, -12.9), turned to 90 degrees
- moved R9 19.1 mm to (4.20, -35.8)
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Connections:
- new net N$1: C30.2, D1.1, R25.2, U7.5
- new net N$2: C31.1, U7.1, U7.3
- new net N$3: C6.1, C8.A, D2.1, FB1.2
- new net N$5: R25.1, R26.2, U7.4
- net 5.0V: now also D1.5, D2.5; no longer C6.1, C8.A, FB1.2
- net DGND: now also C31.2, D1.2, R26.1
- net PGND: now also C30.1, D2.2, U7.2
Routing:
- net CHASSIS: track 531.6 -> 0.00 mm, vias 4 -> 0
- net DGND: track 415.5 -> 0.14 mm, vias 35 -> 0
- net 3.1V: track 281.7 -> 0.00 mm, vias 22 -> 0
- net LOAD_INPUT+: track 145.6 -> 0.00 mm, vias 4 -> 0
- net FEEDBACK: track 140.7 -> 0.00 mm, vias 6 -> 0
- net PGND: track 125.4 -> 0.00 mm, vias 6 -> 0
- net SPI_SCK: track 120.0 -> 0.00 mm, vias 8 -> 0
- net 5.0V: track 117.1 -> 0.00 mm, vias 10 -> 0
- net SHUNT_MID: track 111.8 -> 0.00 mm, vias 3 -> 0
- net SPI_MOSI: track 108.9 -> 0.00 mm, vias 6 -> 0
- net !LCD_CS: track 105.1 -> 0.00 mm, vias 4 -> 0
- net LCD_A0: track 104.3 -> 0.00 mm, vias 6 -> 0
- net !LCD_RST: track 103.8 -> 0.00 mm, vias 4 -> 0
- net FET_GATE: track 91.7 -> 0.00 mm, vias 11 -> 0
- net SHUNT_LOW: track 90.2 -> 0.00 mm, vias 2 -> 0
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
Commit message: Finished Board Layout
Parts:
- removed C30, C31: 1µF 10%, CougsInSpace-Capacitors:1608
- removed D1: LTC4411, CougsInSpace-DiscreteSemi:SOT23-5
- removed J7: 12 V Input, CougsInSpace-Connectors:BARREL-2.1X5.5-R
- removed R25: 10kΩ 0.1%, CougsInSpace-Resistors:1608
- removed R26: 30kΩ 1%, CougsInSpace-Resistors:1608
- removed U7: TPS73250, CougsInSpace-IC-Power:SOT23-5
- added C32, C33: 1µF 10%, CougsInSpace-Capacitors:1608
- added D3: LTC4411, CougsInSpace-DiscreteSemi:SOT23-5
- added J8: 12 V Input, CougsInSpace-Connectors:BARREL-2.1X5.5-R
- added R27: 10kΩ 0.1%, CougsInSpace-Resistors:1608
- added R28: 30kΩ 1%, CougsInSpace-Resistors:1608
- added U8: TPS73250, CougsInSpace-IC-Power:SOT23-5
- moved C1 30.0 mm to (-0.15, -3.85)
- moved J6 27.5 mm to (19.9, -7.95)
- moved C2 19.9 mm to (-2.85, -16.3), turned to 90 degrees
- moved C10 19.6 mm to (12.3, -8.35), turned to 270 degrees
- moved R3 17.9 mm to (-34.1, -11.1)
- moved C29 11.5 mm to (13.1, -20.8)
- moved C11 11.1 mm to (12.3, -15.2), turned to 270 degrees
- moved U6 9.34 mm to (22.3, -17.2), turned to 180 degrees
- moved C27 8.42 mm to (-24.9, -40.8)
- moved U4 8.17 mm to (17.9, -20.5)
- moved C25 7.65 mm to (19.0, -15.2)
- moved U5 7.40 mm to (13.7, -25.1), turned to 180 degrees
- moved C28 6.96 mm to (17.1, -28.6)
- moved C24 5.99 mm to (12.0, -33.0)
- moved R14 3.35 mm to (-3.95, -49.6)
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Connections:
- removed net N$1: C30.2, D1.1, R25.2, U7.5
- removed net N$5: R25.1, R26.2, U7.4
- new net N$4: C32.1, D3.1, R27.2, U8.5
- new net N$7: R27.1, R28.2, U8.4
- net 12.0V: now also J8.1; no longer J7.1
- net 5.0V: now also D3.5; no longer D1.5
- net DGND: no longer C31.2, D1.2, R26.1
- net N$2: now also C33.1, U8.1, U8.3; no longer C31.1, U7.1, U7.3
- net PGND: now also C32.2, C33.2, D3.2, J8.2, J8.3, R28.1, U8.2; no longer C30.1, J7.2, J7.3, U7.2
Routing:
- net DGND: track 0.14 -> 456.8 mm, vias 0 -> 21
- net CHASSIS: track 0.00 -> 398.5 mm
- net PGND: track 0.00 -> 241.3 mm, vias 0 -> 13
- net 3.1V: track 0.00 -> 238.9 mm, vias 0 -> 18
- net FEEDBACK: track 0.00 -> 127.4 mm
- net 12.0V: track 0.00 -> 117.9 mm, vias 0 -> 1
- net 5.0V: track 0.00 -> 106.9 mm, vias 0 -> 3
- net FET_GATE: track 0.00 -> 89.2 mm, vias 0 -> 3
- net ENC_B: track 0.00 -> 83.8 mm, vias 0 -> 4
- net ENC_A: track 0.00 -> 75.7 mm, vias 0 -> 4
- net NICE_BUTTON: track 0.00 -> 74.6 mm, vias 0 -> 4
- net ENC_SW: track 0.00 -> 70.1 mm, vias 0 -> 1
- net !LCD_CS: track 0.00 -> 65.1 mm, vias 0 -> 2
- net !LCD_RST: track 0.00 -> 59.4 mm, vias 0 -> 2
- net SPI_MOSI: track 0.00 -> 58.2 mm, vias 0 -> 1
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- added copper zone on layer 1, net FEEDBACK
- added copper zone on layer 16, net I_ALT+
- added copper zone on layer 16, net I_ALT-
- added copper zone on layer 16, net LOAD_INPUT+
- added copper zone on layer 1, net LOAD_INPUT-
- added copper zone on layer 1, net SHUNT_LOW
- added copper zone on layer 1, net SHUNT_MID

Commit message: Finalized layout and generated mCAD
Parts:
- removed C32, C33: 1µF 10%, CougsInSpace-Capacitors:1608
- removed DS5: Red, CougsInSpace-LEDs:1608-POL
- removed J8: 12 V Input, CougsInSpace-Connectors:BARREL-2.1X5.5-R
- removed R27: 10kΩ 0.1%, CougsInSpace-Resistors:1608
- removed R28: 30kΩ 1%, CougsInSpace-Resistors:1608
- removed TP5: TEST_POINT-THT-1.0, CougsInSpace-Connectors:THT-1.0
- removed U8: TPS73250, CougsInSpace-IC-Power:SOT23-5
- added C30, C31: 1µF 10%, CougsInSpace-Capacitors:1608
- added DS2: Green, CougsInSpace-LEDs:1608-POL
- added J100: SWD, CougsInSpace-Connectors:SMD2.54-1X06-R
- added LOGO1: SIGNATUREJAYSON, CougsInSpace-Aesthetics:SIGN-JAYSON
- added R100: 5mΩ 1%, CougsInSpace-Resistors:1632-KELVIN
- added R25: 0Ω <20mΩ, CougsInSpace-Resistors:1608
- added TP3: TEST_POINT-SMD-C-1.25, CougsInSpace-Connectors:SMD-C-1.25
- added U7: AD8515, CougsInSpace-IC-Amplifiers:SOT23-5
- C11: value 100nF 10% -> 10nF 10%
- C12: value 4.7µF 10% -> 100nF 10%; device CougsInSpace-Capacitors:4028-POL -> CougsInSpace-Capacitors:1608
- C13: value 100nF 10% -> 4.7µF 10%; device CougsInSpace-Capacitors:1608 -> CougsInSpace-Capacitors:4028-POL
- C14, C17, C22: value 1µF 10% -> 100nF 10%
- C16: value 1µF 10% -> 4.7µF 10%; device CougsInSpace-Capacitors:1608 -> CougsInSpace-Capacitors:4028-POL
- C19: value 1nF 1% -> 10pF 5%
- C20: value 1nF 1% -> 100nF 10%
- C23: value 10pF 5% -> 100nF 10%
- C24, C27, C3: value 100nF 10% -> 1µF 10%
- C25, C26: value 100nF 10% -> 1nF 1%
- C4: value 47pF 5% -> 1µF 10%
- C5: value 47pF 5% -> 100nF 10%
- C7: value 10nF 10% -> 47pF 5%
- C8: value 4.7µF 10% -> 47pF 5%; device CougsInSpace-Capacitors:4028-POL -> CougsInSpace-Capacitors:1608
- DS1: value Green -> Red
- J1: value USB -> FAN; device CougsInSpace-Connectors:USB-B-FEMALE -> CougsInSpace-Connectors:THT2.54-1X04-LOCK
- J2: value Load -> 12 V Input; device CougsInSpace-Connectors:TERMINAL_SPRING-02 -> CougsInSpace-Connectors:BARREL-2.1X5.5-R
- J3: value Alternate Current Sense -> USB; device CougsInSpace-Connectors:TERMINAL_SPRING-02 -> CougsInSpace-Connectors:USB-B-FEMALE
- J4: value Voltage Sense -> Load Input; device CougsInSpace-Connectors:TERMINAL_SPRING-03 -> CougsInSpace-Connectors:TERMINAL_SPRING-02
- J5: value SWD -> Voltage Input; device CougsInSpace-Connectors:SMD2.54-1X06-R -> CougsInSpace-Connectors:TERMINAL_SPRING-03
- J6: value FAN -> Auxiliary Current Input; device CougsInSpace-Connectors:THT2.54-1X04-LOCK -> CougsInSpace-Connectors:TERMINAL_SPRING-02
- Q2: value SiRA20DP -> IRFP4368PBF; device CougsInSpace-DiscreteSemi:POWERPAK-SO-8 -> CougsInSpace-DiscreteSemi:TO-247-3-DOWN
- Q4: value IRFP4368PBF -> SiRA20DP; device CougsInSpace-DiscreteSemi:TO-247-3-DOWN -> CougsInSpace-DiscreteSemi:POWERPAK-SO-8
- R1: value 50mΩ 1% -> 10kΩ 0.1%
- R11: value 1kΩ 0.1% -> 0Ω <20mΩ
- R12: value 30kΩ 1% -> 1kΩ 0.1%
- R13: value 1kΩ 0.1% -> 510mΩ 1%
- R14: value 30kΩ 1% -> 50mΩ 1%
- R15: value 1kΩ 0.1% -> 5mΩ 1%; device CougsInSpace-Resistors:1608 -> CougsInSpace-Resistors:1632-KELVIN
- R16: value 10kΩ 0.1% -> 1kΩ 0.1%
- R18: value 0Ω <20mΩ -> 47kΩ 0.1%
- R19: value 0Ω <20mΩ -> 1kΩ 0.1%
- R2: value 5mΩ 1% -> 1kΩ 0.1%; device CougsInSpace-Resistors:1632-KELVIN -> CougsInSpace-Resistors:1608
- R20, R23, R9: value 1kΩ 0.1% -> 10kΩ 0.1%
- R21: value 0Ω <20mΩ -> 30kΩ 1%
- R24: value 10kΩ 0.1% -> 30kΩ 1%
- R3: value 27Ω 1% -> 30kΩ 1%
- R5: value 510mΩ 1% -> 1kΩ 0.1%
- R6: value 5mΩ 1% -> 27Ω 1%; device CougsInSpace-Resistors:1632-KELVIN -> CougsInSpace-Resistors:1608
- R7: value 10kΩ 0.1% -> 0Ω <20mΩ
- R8: value 47kΩ 0.1% -> 1kΩ 0.1%
- SW1: value Nice Knob -> Control Knob
- TP1: value TEST_POINT-SMD-C-1.25 -> TEST_POINT-THT-1.0; device CougsInSpace-Connectors:SMD-C-1.25 -> CougsInSpace-Connectors:THT-1.0
- U1: value STM32L476RGT -> TPS73250; device CougsInSpace-IC-µController:QFP-64-1010 -> CougsInSpace-IC-Power:SOT23-5
- U2: value AD8515 -> STM32L476RGT; device CougsInSpace-IC-Amplifiers:SOT23-5 -> CougsInSpace-IC-µController:QFP-64-1010
- U5: value LP5907MFX-3.1 -> INA199C1; device CougsInSpace-IC-Power:SOT23-5 -> CougsInSpace-IC-Amplifiers:SOT363
- U6: value INA199C1 -> LP5907MFX-3.1; device CougsInSpace-IC-Amplifiers:SOT363 -> CougsInSpace-IC-Power:SOT23-5
- moved J3 85.4 mm to (-44.5, -12.5)
- moved R6 70.5 mm to (-34.1, -13.5), turned to 0 degrees
- moved R2 70.5 mm to (-15.2, -5.25), flipped to the top, turned to 180 degrees
- moved R1 67.9 mm to (-31.1, 3.00), turned to 0 degrees
- moved J1 64.5 mm to (19.9, -7.95)
- moved J6 58.9 mm to (47.4, -60.0), turned to 90 degrees
- moved R15 55.1 mm to (34.8, -28.4), turned to 90 degrees
- moved C17 52.8 mm to (17.8, -24.8), turned to 180 degrees
- moved C25 52.6 mm to (-24.9, -44.2), turned to 180 degrees
- moved R5 49.4 mm to (-19.5, -11.5), turned to 0 degrees
- moved C15 49.4 mm to (13.1, -20.8)
- moved C29 49.4 mm to (-25.0, -52.2)
- moved C5 48.8 mm to (12.3, -8.35)
- moved C26 48.2 mm to (-25.0, -47.0), turned to 0 degrees
- moved Q4 48.2 mm to (34.0, -22.6), turned to 90 degrees
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- renumbered D3 to D1, TP6 to TP2
Connections:
- net !LCD_CS: now also U2.16; no longer U1.16
- net !LCD_RST: now also U2.15; no longer U1.15
- net 12.0V: now also J1.2, J2.1; no longer J6.2, J8.1
- net 3.1V: now also C12.1, C15.1, C17.1, C22.1, C23.1, C5.1, C9.1, DS1.A, DS2.A, R25.1, R8.2, R9.1, U2.1, U2.19, U2.32, U2.48, U2.64, U5.3, U6.5; no longer C10.1, C11.1, C24.1, C26.1, C27.1, C29.1, C3.1, DS3.A, DS5.A, R11.2, R19.1, R7.1, U1.1, U1.19, U1.32, U1.48, U1.64, U5.5, U6.3
- net 5.0V: now also C10.1, C21.1, U6.1, U6.3, U7.5; no longer C25.1, C28.1, U2.5, U5.1, U5.3
- net AGND: now also C16.C, C20.2, R7.1, U2.12; no longer C12.C, C13.2, R17.1, U1.12
- net AVDD: now also C16.A, C20.1, TP3.1, U2.13; no longer C12.A, C13.1, TP1.1, U1.13
- net BOOT0: now also R17.2, U2.60; no longer R10.2, U1.60
- net C1+: now also C25.1; no longer C20.1
- net C1-: now also C25.2; no longer C20.2
- net C2+: now also C26.1; no longer C19.1
- net C2-: now also C26.2; no longer C19.2
- net CBUS1: now also R5.1; no longer R15.1
- net CBUS2: now also R2.1; no longer R13.1
- net CHASSIS: now also J3.SHIELD@1, J3.SHIELD@2, R11.2; no longer J1.SHIELD@1, J1.SHIELD@2, R18.2
- net DGND: now also C12.2, C13.C, C19.2, C24.1, C28.2, C29.2, C30.2, C31.2, C8.2, DS3.C, J100.3, J3.4, R10.2, R17.1, R19.1, R20.1, R7.2, U2.18, U2.31, U2.47, U2.63, U5.1, U5.2, U7.2; no longer C15.2, C16.2, C21.1, C24.2, C25.2, C26.2, C3.2, C4.2, C8.C, DS1.C, J1.4, J5.3, R10.1, R17.2, R21.2, R24.1, R9.1, U1.18, U1.31, U1.47, U1.63, U2.2, U6.1, U6.2
- net ENC_A: now also U2.38; no longer U1.38
- net ENC_B: now also U2.39; no longer U1.39
- net ENC_SW: now also U2.40; no longer U1.40
- net FAN_CONTROL: now also J1.4, U2.22; no longer J6.4, U1.22
- net FAN_SENSE: now also J1.3, U2.44; no longer J6.3, U1.44
- net FEEDBACK: now also Q2.3, Q3.5, Q3.6, Q3.7, Q3.8, Q3.PAD, R13.2, U7.4; no longer Q2.5, Q2.6, Q2.7, Q2.8, Q2.PAD, Q4.3, R5.2, U2.4
- net FET_1: now also Q3.4, U2.25; no longer Q2.4, U1.25
- net FET_2: now also Q4.4, U2.37; no longer Q3.4, U1.37
- net FET_GATE: now also Q2.1, U7.1; no longer Q4.1, U2.1
- net INPUT_SHUNT+: now also R100.2-KELVIN, U5.4; no longer R2.2-KELVIN, U4.4
- net INPUT_SHUNT-: now also R100.1-KELVIN, U5.5; no longer R2.1-KELVIN, U4.5
- net I_ADJ: now also R18.2, U2.20; no longer R8.2, U1.20
- net I_ALT: now also U2.10, U5.6; no longer U1.10, U4.6
- net I_ALT+: now also J6.1, R100.2; no longer J3.1, R2.2
- net I_ALT-: now also J6.2, R100.1; no longer J3.2, R2.1
- net I_LOAD: now also U2.8, U4.6; no longer U1.8, U6.6
- net LCD_A0: now also U2.14; no longer U1.14
- net LCD_LED: now also R25.2; no longer R19.2
- net LCD_V0: now also C31.1; no longer C17.1
- net LCD_V1: now also C30.1; no longer C16.1
- net LCD_V2: now also C29.1; no longer C15.1
- net LCD_V3: now also C28.1; no longer C14.1
- net LCD_V4: now also C27.1; no longer C22.1
- net LOAD_INPUT+: now also J4.1, Q2.2, Q2.PAD; no longer J2.1, Q4.2, Q4.PAD
- net LOAD_INPUT-: now also J4.2, R15.1, R16.2; no longer J2.2, R22.2, R6.1
- net N$2: now also C4.1, U1.1, U1.3; no longer C33.1, U8.1, U8.3
- net N$3: now also C13.A, C14.1; no longer C6.1, C8.A
- net N$4: now also C3.1, R1.2, U1.5; no longer C32.1, R27.2, U8.5
- net N$7: now also R1.1, R3.2, U1.4; no longer R27.1, R28.2, U8.4
- net NICE_BUTTON: now also U2.52; no longer U1.52
- net NRST: now also J100.5, U2.7; no longer J5.5, U1.7
- net OP_AMP_IN: now also R18.1, R19.2, U7.3; no longer R8.1, R9.2, U2.3
- net OSC_IN: now also C19.1, U2.5; no longer C23.1, U1.5
- net OSC_OUT: now also U2.6; no longer U1.6
- net OUTPUT_SHUNT+: now also R15.2-KELVIN, U4.4; no longer R6.2-KELVIN, U6.4
- net OUTPUT_SHUNT-: now also R15.1-KELVIN, U4.5; no longer R6.1-KELVIN, U6.5
- net PGND: now also C15.2, C21.2, C3.2, C4.2, J1.1, J2.2, J2.3, R10.1, R11.1, R3.1, U1.2, U6.2; no longer C28.2, C29.2, C32.2, C33.2, J6.1, J8.2, J8.3, R18.1, R21.1, R28.1, U5.2, U8.2
- net RX: now also U2.43; no longer U1.43
- net RXLED_C: now also DS1.C, R2.2; no longer DS5.C, R13.2
- net SHUNT_LOW: now also Q4.1, Q4.2, Q4.3, R14.1, R15.2; no longer Q3.1, Q3.2, Q3.3, R1.1, R6.2
- net SHUNT_MID: now also Q3.1, Q3.2, Q3.3, Q4.5, Q4.6, Q4.7, Q4.8, Q4.PAD, R13.1, R14.2; no longer Q2.1, Q2.2, Q2.3, Q3.5, Q3.6, Q3.7, Q3.8, Q3.PAD, R1.2, R5.1
- net SPI_MOSI: now also U2.23; no longer U1.23
- net SPI_SCK: now also U2.21; no longer U1.21
- net SWCLK: now also J100.2, U2.49; no longer J5.2, U1.49
- net SWDIO: now also J100.4, U2.46; no longer J5.4, U1.46
- net SWO: now also J100.6, U2.55; no longer J5.6, U1.55
- net TO_LED: now also R12.2, U2.54; no longer R20.2, U1.54
- net TO_LED_ANODE: now also DS3.A, R12.1; no longer DS1.A, R20.1
- net TX: now also U2.42; no longer U1.42
- net TXLED_C: now also DS2.C, R5.2; no longer DS3.C, R15.2
- net USB5V: now also C11.1, J3.1, TP1.1; no longer C7.1, J1.1, TP5.1
- net USB_CONN_N: now also C8.1, J3.2, R6.1; no longer C4.1, J1.2, R4.1
- net USB_CONN_P: now also C7.1, J3.3, R4.1; no longer C5.1, J1.3, R3.1
- net USB_N: now also R6.2; no longer R4.2
- net USB_P: now also R4.2; no longer R3.2
- net USB_RESET: now also C6.1, R9.2; no longer C9.1, R7.2
- net VOUT: now also C24.2; no longer C21.2
- net VSENSE: now also J100.1, R8.1; no longer J5.1, R11.1
- net VSENSE_ALT: now also J5.1, R21.2; no longer J4.1, R14.2
- net VSENSE_GND: now also J5.3, R22.2; no longer J4.3, R23.2
- net VSENSE_LOAD: now also J5.2, R24.2; no longer J4.2, R12.2
- net V_ALT: now also R20.2, R21.1, U2.9; no longer R14.1, R24.2, U1.9
- net V_LOAD: now also R23.2, R24.1, U2.11; no longer R12.1, R16.2, U1.11
Routing:
- net LOAD_INPUT+: track 18.3 -> 155.4 mm
- net FEEDBACK: track 127.4 -> 81.9 mm
- net DGND: track 456.8 -> 479.7 mm, vias 21 -> 25
- net INPUT_SHUNT+: track 38.1 -> 58.3 mm
- net INPUT_SHUNT-: track 39.7 -> 57.0 mm
- net VSENSE_ALT: track 28.8 -> 11.9 mm
- net VSENSE_GND: track 12.9 -> 27.8 mm
- net AVDD: track 53.1 -> 38.8 mm
- net LOAD_INPUT-: track 24.0 -> 13.3 mm
- net TXLED_C: track 11.3 -> 1.50 mm, vias 2 -> 0
- net VSENSE: track 30.2 -> 39.8 mm
- net FET_GATE: track 89.2 -> 98.0 mm
- net NRST: track 36.5 -> 44.2 mm
- net SWO: track 30.4 -> 37.8 mm
- net SWDIO: track 47.6 -> 54.6 mm
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- added copper zone on layer 16, net CHASSIS
- added copper zone on layer 1, net DGND
- added copper zone on layer 16, net DGND
Other:
- board text added: "Electronic Load V1.0"
- board text added: "RX"
- board text added: "TX"
