File: Subsystems/Electronics/Testing/battery-charger/ElectricalDesign/untitled.sch (EAGLE design)
At the start: 1 part

Commit message: updated schematics
Parts:
- removed RN1: 10kΩ 1%, CougsInSpace-Resistors:RES-4-H-10K-1632
Changed lines of the file:
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@@
 </classes>
 <parts>
-<part name="RN1" library="CougsInSpace-Resistors" deviceset="RES-4-H" device="-1632" technology="-10K" value="10kΩ 1%"/>
+<part name="FRAME1" library="CougsInSpace-Aesthetics" deviceset="FRAME-A" device=""/>
 </parts>
 <sheets>
@@
 </plain>
 <instances>
-<instance part="RN1" gate="A" x="43.18" y="43.18" smashed="yes">
-<attribute name="NAME" x="41.91" y="45.212" size="1.27" layer="95" align="center"/>
-<attribute name="VALUE" x="41.656" y="41.148" size="1.27" layer="96" align="center-right"/>
-<attribute name="PACKAGE" x="41.656" y="39.624" size="1.27" layer="97" align="center-right"/>
-<attribute name="POWER" x="42.164" y="41.148" size="1.27" layer="97" align="center-left"/>
-<attribute name="TEMP" x="42.164" y="39.624" size="1.27" layer="97" align="center-left"/>
-<attribute name="SKU" x="41.91" y="38.1" size="1.27" layer="97" align="center"/>
+<instance part="FRAME1" gate="G$1" x="-38.1" y="10.16" smashed="yes">
+<attribute name="LAST_DATE_TIME" x="189.23" y="11.43" size="3.81" layer="94" ratio="15" align="bottom-right"/>
+<attribute name="SHEET" x="219.71" y="11.43" size="3.81" layer="94" ratio="15" align="bottom-right"/>
 </instance>
 </instances>
@@
 </schematic>
 </drawing>
+<compatibility>
+<note version="6.3" minversion="6.2.2" severity="warning">
+Since Version 6.2.2 text objects can contain more than one line,
+which will not be processed correctly with this version.
+</note>
+</compatibility>
 </eagle>
